File: doc/kicad/fm02-mb-1/FM02-MB-1/FM02-MB-1.sch (KiCad schematic (older format))
At the start: 16 parts, among them J1 Conn_01x04, J2 Conn_01x06, Q1 Q_NMOS_DGS, Q2 Q_NMOS_DGS, Q3 Q_NMOS_DGS, Q4 Q_NMOS_DGS, U1 MPU-6050

Commit message: doc/kicad: FM02-MB-1 v0.1
Parts:
- removed Q1, Q2, Q3, Q4: Q_NMOS_DGS, Package_TO_SOT_SMD:TO-252-3_TabPin2, symbol Device:Q_NMOS_DGS
- added Q1, Q2, Q3, Q4: Q_NMOS_DSG, Package_TO_SOT_SMD:TO-252-2, symbol Device:Q_NMOS_DSG
- JM1, JM2, JM3, JM4: footprint Connector_SMD:CSMD-JM1P -> Connector_SMD:CSMD-JM2
Connections:
- net +BATT: now also Q1.1 (D), Q2.1 (D), Q3.1 (D), Q4.1 (D)
- net M1: now also Q1.2 (S)
- net M2: now also Q2.2 (S)
- net M3: now also Q3.2 (S)
- net M4: now also Q4.2 (S)
- net QC1: now also Q1.3 (G)
- net QC2: now also Q2.3 (G)
- net QC3: now also Q3.3 (G)
- net QC4: now also Q4.3 (G)
- net SCL1: now also J2.6 (Pin_6); no longer J2.5 (Pin_5)
- net SDA1: now also J2.5 (Pin_5); no longer J2.6 (Pin_6)
Changed lines of the file:
@@
-	1    0    0    -1
-$EndComp
-$Comp
-L Device:Q_NMOS_DGS Q1
-U 1 1 5F8C37E1
-P 1900 5000
-F 0 "Q1" H 2104 5046 50  0000 L CNN
-F 1 "Q_NMOS_DGS" H 2104 4955 50  0000 L CNN
-F 2 "Package_TO_SOT_SMD:TO-252-3_TabPin2" H 2100 5100 50  0001 C CNN
-F 3 "~" H 1900 5000 50  0001 C CNN
-	1    1900 5000
-	1    0    0    -1
-$EndComp
-$Comp
-L Device:Q_NMOS_DGS Q2
-U 1 1 5F8C3CDC
-P 3900 5000
-F 0 "Q2" H 4104 5046 50  0000 L CNN
-F 1 "Q_NMOS_DGS" H 4104 4955 50  0000 L CNN
-F 2 "Package_TO_SOT_SMD:TO-252-3_TabPin2" H 4100 5100 50  0001 C CNN
-F 3 "~" H 3900 5000 50  0001 C CNN
-	1    3900 5000
-	1    0    0    -1
-$EndComp
-$Comp
-L Device:Q_NMOS_DGS Q3
-U 1 1 5F8C42D7
-P 5900 5000
-F 0 "Q3" H 6104 5046 50  0000 L CNN
-F 1 "Q_NMOS_DGS" H 6104 4955 50  0000 L CNN
-F 2 "Package_TO_SOT_SMD:TO-252-3_TabPin2" H 6100 5100 50  0001 C CNN
-F 3 "~" H 5900 5000 50  0001 C CNN
-	1    5900 5000
-	1    0    0    -1
-$EndComp
-$Comp
-L Device:Q_NMOS_DGS Q4
-U 1 1 5F8C48F1
-P 7900 5000
-F 0 "Q4" H 8104 5046 50  0000 L CNN
-F 1 "Q_NMOS_DGS" H 8104 4955 50  0000 L CNN
-F 2 "Package_TO_SOT_SMD:TO-252-3_TabPin2" H 8100 5100 50  0001 C CNN
-F 3 "~" H 7900 5000 50  0001 C CNN
-	1    7900 5000
 	1    0    0    -1
 $EndComp
@@
 F 0 "JM1" V 1872 5780 50  0000 L CNN
 F 1 "Conn_01x01" V 1963 5780 50  0000 L CNN
-F 2 "Connector_SMD:CSMD-JM1P" H 2000 5700 50  0001 C CNN
+F 2 "Connector_SMD:CSMD-JM2" H 2000 5700 50  0001 C CNN
 F 3 "~" H 2000 5700 50  0001 C CNN
 	1    2000 5700
@@
 F 0 "JM2" V 3872 5780 50  0000 L CNN
 F 1 "Conn_01x01" V 3963 5780 50  0000 L CNN
-F 2 "Connector_SMD:CSMD-JM1P" H 4000 5700 50  0001 C CNN
+F 2 "Connector_SMD:CSMD-JM2" H 4000 5700 50  0001 C CNN
 F 3 "~" H 4000 5700 50  0001 C CNN
 	1    4000 5700
@@
 F 0 "JM3" V 5872 5780 50  0000 L CNN
 F 1 "Conn_01x01" V 5963 5780 50  0000 L CNN
-F 2 "Connector_SMD:CSMD-JM1P" H 6000 5700 50  0001 C CNN
+F 2 "Connector_SMD:CSMD-JM2" H 6000 5700 50  0001 C CNN
 F 3 "~" H 6000 5700 50  0001 C CNN
 	1    6000 5700
@@
 F 0 "JM4" V 7872 5780 50  0000 L CNN
 F 1 "Conn_01x01" V 7963 5780 50  0000 L CNN
-F 2 "Connector_SMD:CSMD-JM1P" H 8000 5700 50  0001 C CNN
+F 2 "Connector_SMD:CSMD-JM2" H 8000 5700 50  0001 C CNN
 F 3 "~" H 8000 5700 50  0001 C CNN
 	1    8000 5700
@@
 Text Label 4800 1800 2    50   ~ 0
 LED2
+Wire Wire Line
+	4550 1700 4800 1700
+$Comp
+L Device:Q_NMOS_DSG Q1
+U 1 1 5F9434BD
+P 1900 5000
+F 0 "Q1" H 2104 5046 50  0000 L CNN
+F 1 "Q_NMOS_DSG" H 2104 4955 50  0000 L CNN
+F 2 "Package_TO_SOT_SMD:TO-252-2" H 2100 5100 50  0001 C CNN
+F 3 "~" H 1900 5000 50  0001 C CNN
+	1    1900 5000
+	1    0    0    -1
+$EndComp
+$Comp
+L Device:Q_NMOS_DSG Q2
+U 1 1 5F944061
+P 3900 5000
+F 0 "Q2" H 4104 5046 50  0000 L CNN
+F 1 "Q_NMOS_DSG" H 4104 4955 50  0000 L CNN
+F 2 "Package_TO_SOT_SMD:TO-252-2" H 4100 5100 50  0001 C CNN
+F 3 "~" H 3900 5000 50  0001 C CNN
+	1    3900 5000
+	1    0    0    -1
+$EndComp
+$Comp
+L Device:Q_NMOS_DSG Q3
+U 1 1 5F944564
+P 5900 5000
+F 0 "Q3" H 6104 5046 50  0000 L CNN
+F 1 "Q_NMOS_DSG" H 6104 4955 50  0000 L CNN
+F 2 "Package_TO_SOT_SMD:TO-252-2" H 6100 5100 50  0001 C CNN
+F 3 "~" H 5900 5000 50  0001 C CNN
+	1    5900 5000
+	1    0    0    -1
+$EndComp
+$Comp
+L Device:Q_NMOS_DSG Q4
+U 1 1 5F944B4E
+P 7900 5000
+F 0 "Q4" H 8104 5046 50  0000 L CNN
+F 1 "Q_NMOS_DSG" H 8104 4955 50  0000 L CNN
+F 2 "Package_TO_SOT_SMD:TO-252-2" H 8100 5100 50  0001 C CNN
+F 3 "~" H 7900 5000 50  0001 C CNN
+	1    7900 5000
+	1    0    0    -1
+$EndComp
 Text Label 4800 1900 2    50   ~ 0
+SDA1
+Text Label 4800 2000 2    50   ~ 0
 SCL1
-Text Label 4800 2000 2    50   ~ 0
-SDA1
-Wire Wire Line
-	4550 1700 4800 1700
 $EndSCHEMATC
