File: doc/kicad/fm01-es2-1/FM01-ES2-1/FM01-ES2-1.sch (KiCad schematic (older format))
At the start: 27 parts, among them J1 USB_B_Micro, J2 Conn_01x10, J3 Conn_01x10, J4 Conn_01x30, U1 ESP32-S2-WROVER-I

Commit message: doc/kicad: FM01-ES2-1  add PCB
Parts:
- C1, C10, C11, C2, C3, C4: footprint (none) -> Capacitor_SMD:C_0402_1005Metric
- D1, D2: footprint (none) -> LED_SMD:LED_0402_1005Metric
- J1: footprint (none) -> Connector_USB:USB_Micro-B_Molex_47346-0001
- J2, J3: footprint (none) -> Connector_Hirose:Hirose_DF13C_CL535-0410-4-51_1x10-1MP_P1.25mm_Vertical
- J4: footprint (none) -> Connector_FFC-FPC:Hirose_FH12-30S-0.5SH_1x30-1MP_P0.50mm_Horizontal
- R1, R10, R11, R18, R2, R3, R30, R31, R32, R33, R34, R35, R36, R4: footprint (none) -> Resistor_SMD:R_0402_1005Metric
Changed lines of the file:
@@
 EN
 $Comp
-L power:+3.3V #PWR?
+L power:+3.3V #PWR0101
 U 1 1 5F98722A
 P 1000 1000
-F 0 "#PWR?" H 1000 850 50  0001 C CNN
+F 0 "#PWR0101" H 1000 850 50  0001 C CNN
 F 1 "+3.3V" H 1015 1173 50  0000 C CNN
 F 2 "" H 1000 1000 50  0001 C CNN
@@
 F 0 "C1" H 1115 1396 50  0000 L CNN
 F 1 "22u" H 1115 1305 50  0000 L CNN
-F 2 "" H 1038 1200 50  0001 C CNN
+F 2 "Capacitor_SMD:C_0402_1005Metric" H 1038 1200 50  0001 C CNN
 F 3 "~" H 1000 1350 50  0001 C CNN
 	1    1000 1350
@@
 F 0 "C2" H 1615 1396 50  0000 L CNN
 F 1 "0.1u" H 1615 1305 50  0000 L CNN
-F 2 "" H 1538 1200 50  0001 C CNN
+F 2 "Capacitor_SMD:C_0402_1005Metric" H 1538 1200 50  0001 C CNN
 F 3 "~" H 1500 1350 50  0001 C CNN
 	1    1500 1350
@@
 $EndComp
 $Comp
-L power:GND #PWR?
+L power:GND #PWR0102
 U 1 1 5F987CC2
 P 1000 1600
-F 0 "#PWR?" H 1000 1350 50  0001 C CNN
+F 0 "#PWR0102" H 1000 1350 50  0001 C CNN
 F 1 "GND" H 1005 1427 50  0000 C CNN
 F 2 "" H 1000 1600 50  0001 C CNN
@@
 $EndComp
 $Comp
-L power:GND #PWR?
+L power:GND #PWR0103
 U 1 1 5F987E94
 P 1500 1600
-F 0 "#PWR?" H 1500 1350 50  0001 C CNN
+F 0 "#PWR0103" H 1500 1350 50  0001 C CNN
 F 1 "GND" H 1505 1427 50  0000 C CNN
 F 2 "" H 1500 1600 50  0001 C CNN
@@
 $EndComp
 $Comp
-L power:PWR_FLAG #FLG?
+L power:PWR_FLAG #FLG0101
 U 1 1 5F98867E
 P 1000 1150
-F 0 "#FLG?" H 1000 1225 50  0001 C CNN
+F 0 "#FLG0101" H 1000 1225 50  0001 C CNN
 F 1 "PWR_FLAG" V 1000 1277 50  0000 L CNN
 F 2 "" H 1000 1150 50  0001 C CNN
@@
 	0    -1   -1   0
 $EndComp
-$Comp
-L power:PWR_FLAG #FLG?
-U 1 1 5F9888C9
-P 1000 1500
-F 0 "#FLG?" H 1000 1575 50  0001 C CNN
-F 1 "PWR_FLAG" V 1000 1627 50  0000 L CNN
-F 2 "" H 1000 1500 50  0001 C CNN
-F 3 "~" H 1000 1500 50  0001 C CNN
-	1    1000 1500
-	0    -1   -1   0
-$EndComp
 Wire Wire Line
 	1500 1200 1500 1150
@@
 Wire Wire Line
 	1000 1500 1000 1600
-Connection ~ 1000 1500
 Wire Wire Line
 	1500 1500 1500 1600
@@
 GND
 $Comp
-L power:GND #PWR?
+L power:GND #PWR0104
 U 1 1 5F98E86E
 P 5500 4600
-F 0 "#PWR?" H 5500 4350 50  0001 C CNN
+F 0 "#PWR0104" H 5500 4350 50  0001 C CNN
 F 1 "GND" H 5505 4427 50  0000 C CNN
 F 2 "" H 5500 4600 50  0001 C CNN
@@
 F 0 "R3" V 4293 2500 50  0000 C CNN
 F 1 "10k" V 4384 2500 50  0000 C CNN
-F 2 "" V 4430 2500 50  0001 C CNN
+F 2 "Resistor_SMD:R_0402_1005Metric" V 4430 2500 50  0001 C CNN
 F 3 "~" H 4500 2500 50  0001 C CNN
 	1    4500 2500
@@
 F 0 "C3" H 4815 2346 50  0000 L CNN
 F 1 "0.1u" H 4815 2255 50  0000 L CNN
-F 2 "" H 4738 2150 50  0001 C CNN
+F 2 "Capacitor_SMD:C_0402_1005Metric" H 4738 2150 50  0001 C CNN
 F 3 "~" H 4700 2300 50  0001 C CNN
 	1    4700 2300
@@
 $EndComp
 $Comp
-L power:GND #PWR?
+L power:GND #PWR0105
 U 1 1 5F98FC02
 P 4700 2150
-F 0 "#PWR?" H 4700 1900 50  0001 C CNN
+F 0 "#PWR0105" H 4700 1900 50  0001 C CNN
 F 1 "GND" H 4705 1977 50  0000 C CNN
 F 2 "" H 4700 2150 50  0001 C CNN
@@
 F 0 "R1" H 1070 2696 50  0000 L CNN
 F 1 "15" H 1070 2605 50  0000 L CNN
-F 2 "" V 930 2650 50  0001 C CNN
+F 2 "Resistor_SMD:R_0402_1005Metric" V 930 2650 50  0001 C CNN
 F 3 "~" H 1000 2650 50  0001 C CNN
 	1    1000 2650
@@
 F 0 "R2" H 1570 2696 50  0000 L CNN
 F 1 "15" H 1570 2605 50  0000 L CNN
-F 2 "" V 1430 2650 50  0001 C CNN
+F 2 "Resistor_SMD:R_0402_1005Metric" V 1430 2650 50  0001 C CNN
 F 3 "~" H 1500 2650 50  0001 C CNN
 	1    1500 2650
@@
 F 0 "D1" V 1039 2832 50  0000 R CNN
 F 1 "LED-G" V 948 2832 50  0000 R CNN
-F 2 "" H 1000 2950 50  0001 C CNN
+F 2 "LED_SMD:LED_0402_1005Metric" H 1000 2950 50  0001 C CNN
 F 3 "~" H 1000 2950 50  0001 C CNN
 	1    1000 2950
@@
 F 0 "D2" V 1539 2832 50  0000 R CNN
 F 1 "LED-B" V 1448 2832 50  0000 R CNN
-F 2 "" H 1500 2950 50  0001 C CNN
+F 2 "LED_SMD:LED_0402_1005Metric" H 1500 2950 50  0001 C CNN
 F 3 "~" H 1500 2950 50  0001 C CNN
 	1    1500 2950
@@
 $EndComp
 $Comp
-L power:GND #PWR?
+L power:GND #PWR0106
 U 1 1 5F991E18
 P 1000 3100
-F 0 "#PWR?" H 1000 2850 50  0001 C CNN
+F 0 "#PWR0106" H 1000 2850 50  0001 C CNN
 F 1 "GND" H 1005 2927 50  0000 C CNN
 F 2 "" H 1000 3100 50  0001 C CNN
@@
 F 0 "J2" H 3668 3517 50  0000 C CNN
 F 1 "Conn_01x10" H 3668 3426 50  0000 C CNN
-F 2 "" H 3750 2900 50  0001 C CNN
+F 2 "Connector_Hirose:Hirose_DF13C_CL535-0410-4-51_1x10-1MP_P1.25mm_Vertical" H 3750 2900 50  0001 C CNN
 F 3 "~" H 3750 2900 50  0001 C CNN
 	1    3750 2900
@@
 F 0 "J3" H 3368 4717 50  0000 C CNN
 F 1 "Conn_01x10" H 3368 4626 50  0000 C CNN
-F 2 "" H 3450 4100 50  0001 C CNN
+F 2 "Connector_Hirose:Hirose_DF13C_CL535-0410-4-51_1x10-1MP_P1.25mm_Vertical" H 3450 4100 50  0001 C CNN
 F 3 "~" H 3450 4100 50  0001 C CNN
 	1    3450 4100
@@
 F 0 "J4" H 8880 3592 50  0000 L CNN
 F 1 "Conn_01x30" H 8880 3501 50  0000 L CNN
-F 2 "" H 8800 3600 50  0001 C CNN
+F 2 "Connector_FFC-FPC:Hirose_FH12-30S-0.5SH_1x30-1MP_P0.50mm_Horizontal" H 8800 3600 50  0001 C CNN
 F 3 "~" H 8800 3600 50  0001 C CNN
 	1    8800 3600
@@
 F 0 "J1" H 7320 4089 50  0000 R CNN
 F 1 "USB_B_Micro" H 7320 3998 50  0000 R CNN
-F 2 "" H 7700 4050 50  0001 C CNN
+F 2 "Connector_USB:USB_Micro-B_Molex_47346-0001" H 7700 4050 50  0001 C CNN
 F 3 "~" H 7700 4050 50  0001 C CNN
 	1    7550 4100
@@
 F 0 "R18" V 4957 4750 50  0000 C CNN
 F 1 "10k" V 4866 4750 50  0000 C CNN
-F 2 "" V 4680 4750 50  0001 C CNN
+F 2 "Resistor_SMD:R_0402_1005Metric" V 4680 4750 50  0001 C CNN
 F 3 "~" H 4750 4750 50  0001 C CNN
 	1    4750 4750
@@
 F 0 "R4" V 6293 2000 50  0000 C CNN
 F 1 "0" V 6384 2000 50  0000 C CNN
-F 2 "" V 6430 2000 50  0001 C CNN
+F 2 "Resistor_SMD:R_0402_1005Metric" V 6430 2000 50  0001 C CNN
 F 3 "~" H 6500 2000 50  0001 C CNN
 	1    6500 2000
@@
 F 0 "C4" V 6798 2000 50  0000 C CNN
 F 1 "0.1u" V 6889 2000 50  0000 C CNN
-F 2 "" H 7088 1850 50  0001 C CNN
+F 2 "Capacitor_SMD:C_0402_1005Metric" H 7088 1850 50  0001 C CNN
 F 3 "~" H 7050 2000 50  0001 C CNN
 	1    7050 2000
@@
 $EndComp
 $Comp
-L power:GND #PWR?
+L power:GND #PWR0107
 U 1 1 5F9B4FC2
 P 7200 2000
-F 0 "#PWR?" H 7200 1750 50  0001 C CNN
+F 0 "#PWR0107" H 7200 1750 50  0001 C CNN
 F 1 "GND" V 7205 1872 50  0000 R CNN
 F 2 "" H 7200 2000 50  0001 C CNN
@@
 F 0 "R11" V 6393 4100 50  0000 C CNN
 F 1 "0" V 6484 4100 50  0000 C CNN
-F 2 "" V 6530 4100 50  0001 C CNN
+F 2 "Resistor_SMD:R_0402_1005Metric" V 6530 4100 50  0001 C CNN
 F 3 "~" H 6600 4100 50  0001 C CNN
 	1    6600 4100
@@
 F 0 "R10" V 6700 4200 50  0000 C CNN
 F 1 "0" V 6800 4200 50  0000 C CNN
-F 2 "" V 6530 4200 50  0001 C CNN
+F 2 "Resistor_SMD:R_0402_1005Metric" V 6530 4200 50  0001 C CNN
 F 3 "~" H 6600 4200 50  0001 C CNN
 	1    6600 4200
@@
 NoConn ~ 7250 4300
 $Comp
-L power:GND #PWR?
+L power:GND #PWR0108
 U 1 1 5F9C61BB
 P 7550 4500
-F 0 "#PWR?" H 7550 4250 50  0001 C CNN
+F 0 "#PWR0108" H 7550 4250 50  0001 C CNN
 F 1 "GND" H 7555 4327 50  0000 C CNN
 F 2 "" H 7550 4500 50  0001 C CNN
@@
 F 0 "C11" H 6915 3896 50  0000 L CNN
 F 1 "20p" H 6915 3805 50  0000 L CNN
-F 2 "" H 6838 3700 50  0001 C CNN
+F 2 "Capacitor_SMD:C_0402_1005Metric" H 6838 3700 50  0001 C CNN
 F 3 "~" H 6800 3850 50  0001 C CNN
 	1    6800 3850
@@
 F 0 "C10" H 6915 4496 50  0000 L CNN
 F 1 "20p" H 6915 4405 50  0000 L CNN
-F 2 "" H 6838 4300 50  0001 C CNN
+F 2 "Capacitor_SMD:C_0402_1005Metric" H 6838 4300 50  0001 C CNN
 F 3 "~" H 6800 4450 50  0001 C CNN
 	1    6800 4450
@@
 	6800 4200 7250 4200
 $Comp
-L power:GND #PWR?
+L power:GND #PWR0109
 U 1 1 5F9C8F6F
 P 6800 3700
-F 0 "#PWR?" H 6800 3450 50  0001 C CNN
+F 0 "#PWR0109" H 6800 3450 50  0001 C CNN
 F 1 "GND" H 6805 3527 50  0000 C CNN
 F 2 "" H 6800 3700 50  0001 C CNN
@@
 $EndComp
 $Comp
-L power:GND #PWR?
+L power:GND #PWR0110
 U 1 1 5F9C94EE
 P 6800 4600
-F 0 "#PWR?" H 6800 4350 50  0001 C CNN
+F 0 "#PWR0110" H 6800 4350 50  0001 C CNN
 F 1 "GND" H 6805 4427 50  0000 C CNN
 F 2 "" H 6800 4600 50  0001 C CNN
@@
 IO15
 $Comp
-L power:GND #PWR?
+L power:GND #PWR0111
 U 1 1 5F9F66AA
 P 1000 4000
-F 0 "#PWR?" H 1000 3750 50  0001 C CNN
+F 0 "#PWR0111" H 1000 3750 50  0001 C CNN
 F 1 "GND" V 1005 3872 50  0000 R CNN
 F 2 "" H 1000 4000 50  0001 C CNN
@@
 $EndComp
 $Comp
-L power:GND #PWR?
+L power:GND #PWR0112
 U 1 1 5F9F6AE7
 P 1000 4500
-F 0 "#PWR?" H 1000 4250 50  0001 C CNN
+F 0 "#PWR0112" H 1000 4250 50  0001 C CNN
 F 1 "GND" V 1005 4372 50  0000 R CNN
 F 2 "" H 1000 4500 50  0001 C CNN
@@
 F 0 "R30" V 1357 4000 50  0000 C CNN
 F 1 "1k" V 1266 4000 50  0000 C CNN
-F 2 "" V 1080 4000 50  0001 C CNN
+F 2 "Resistor_SMD:R_0402_1005Metric" V 1080 4000 50  0001 C CNN
 F 3 "~" H 1150 4000 50  0001 C CNN
 	1    1150 4000
@@
 F 0 "R31" V 1243 4000 50  0000 C CNN
 F 1 "1k" V 1334 4000 50  0000 C CNN
-F 2 "" V 1380 4000 50  0001 C CNN
+F 2 "Resistor_SMD:R_0402_1005Metric" V 1380 4000 50  0001 C CNN
 F 3 "~" H 1450 4000 50  0001 C CNN
 	1    1450 4000
@@
 F 0 "R32" V 1543 4000 50  0000 C CNN
 F 1 "1k" V 1634 4000 50  0000 C CNN
-F 2 "" V 1680 4000 50  0001 C CNN
+F 2 "Resistor_SMD:R_0402_1005Metric" V 1680 4000 50  0001 C CNN
 F 3 "~" H 1750 4000 50  0001 C CNN
 	1    1750 4000
@@
 F 0 "R33" V 943 4500 50  0000 C CNN
 F 1 "1k" V 1034 4500 50  0000 C CNN
-F 2 "" V 1080 4500 50  0001 C CNN
+F 2 "Resistor_SMD:R_0402_1005Metric" V 1080 4500 50  0001 C CNN
 F 3 "~" H 1150 4500 50  0001 C CNN
 	1    1150 4500
@@
 F 0 "R34" V 1243 4500 50  0000 C CNN
 F 1 "10k" V 1334 4500 50  0000 C CNN
-F 2 "" V 1380 4500 50  0001 C CNN
+F 2 "Resistor_SMD:R_0402_1005Metric" V 1380 4500 50  0001 C CNN
 F 3 "~" H 1450 4500 50  0001 C CNN
 	1    1450 4500
@@
 F 0 "R36" V 1850 4150 50  0000 C CNN
 F 1 "0" V 1950 4150 50  0000 C CNN
-F 2 "" V 1680 4150 50  0001 C CNN
+F 2 "Resistor_SMD:R_0402_1005Metric" V 1680 4150 50  0001 C CNN
 F 3 "~" H 1750 4150 50  0001 C CNN
 	1    1750 4150
@@
 F 0 "R35" V 1550 4650 50  0000 C CNN
 F 1 "0" V 1650 4650 50  0000 C CNN
-F 2 "" V 1380 4650 50  0001 C CNN
+F 2 "Resistor_SMD:R_0402_1005Metric" V 1380 4650 50  0001 C CNN
 F 3 "~" H 1450 4650 50  0001 C CNN
 	1    1450 4650

Commit message: doc/kicad: FM01-ES2-1  add README.md
Parts:
- added R50, R51, R52: 1k, symbol Device:R
- added R53: 0, symbol Device:R
Connections:
- net GND: now also R50.2
- net IO12: now also R53.1
- net VBUS: now reaches J1.1 (VBUS)
- net VBUS: now also R52.1
- new net: R50.1, R51.2, R53.2
- new net: R51.1, R52.2
- no-connect marks 4 -> 3
Other:
- moved on the sheet: J1, R33, R34, R35
Changed lines of the file:
@@
 Sheet 1 1
 Title "FM01-ES2-1"
-Date "2020-10-27"
+Date "2020-10-31"
 Rev "v0.1"
 Comp "sceext"
@@
 L Connector:USB_B_Micro J1
 U 1 1 5F99B066
-P 7550 4100
-F 0 "J1" H 7320 4089 50  0000 R CNN
-F 1 "USB_B_Micro" H 7320 3998 50  0000 R CNN
-F 2 "Connector_USB:USB_Micro-B_Molex_47346-0001" H 7700 4050 50  0001 C CNN
-F 3 "~" H 7700 4050 50  0001 C CNN
-	1    7550 4100
+P 7600 4100
+F 0 "J1" H 7370 4089 50  0000 R CNN
+F 1 "USB_B_Micro" H 7370 3998 50  0000 R CNN
+F 2 "Connector_USB:USB_Micro-B_Molex_47346-0001" H 7750 4050 50  0001 C CNN
+F 3 "~" H 7750 4050 50  0001 C CNN
+	1    7600 4100
 	-1   0    0    -1
 $EndComp
@@
 Wire Wire Line
 	6100 4200 6450 4200
-Text Label 7250 4100 2    50   ~ 0
+Text Label 7300 4100 2    50   ~ 0
 USB_D1+
-Text Label 7250 4200 2    50   ~ 0
+Text Label 7300 4200 2    50   ~ 0
 USB_D1-
 Wire Wire Line
@@
 Wire Wire Line
 	6750 4200 6800 4200
-NoConn ~ 7250 3900
-NoConn ~ 7250 4300
+NoConn ~ 7300 4300
 $Comp
 L power:GND #PWR0108
 U 1 1 5F9C61BB
-P 7550 4500
-F 0 "#PWR0108" H 7550 4250 50  0001 C CNN
-F 1 "GND" H 7555 4327 50  0000 C CNN
-F 2 "" H 7550 4500 50  0001 C CNN
-F 3 "" H 7550 4500 50  0001 C CNN
-	1    7550 4500
-	1    0    0    -1
-$EndComp
-Wire Wire Line
-	7650 4500 7550 4500
-Connection ~ 7550 4500
+P 7600 4500
+F 0 "#PWR0108" H 7600 4250 50  0001 C CNN
+F 1 "GND" H 7605 4327 50  0000 C CNN
+F 2 "" H 7600 4500 50  0001 C CNN
+F 3 "" H 7600 4500 50  0001 C CNN
+	1    7600 4500
+	1    0    0    -1
+$EndComp
+Wire Wire Line
+	7700 4500 7600 4500
+Connection ~ 7600 4500
 $Comp
 L Device:C C11
@@
 Wire Wire Line
 	6800 4000 6800 4100
-Connection ~ 6800 4100
-Wire Wire Line
-	6800 4100 7250 4100
 Wire Wire Line
 	6800 4300 6800 4200
-Connection ~ 6800 4200
-Wire Wire Line
-	6800 4200 7250 4200
 $Comp
 L power:GND #PWR0109
@@
 L power:GND #PWR0112
 U 1 1 5F9F6AE7
-P 1000 4500
-F 0 "#PWR0112" H 1000 4250 50  0001 C CNN
-F 1 "GND" V 1005 4372 50  0000 R CNN
-F 2 "" H 1000 4500 50  0001 C CNN
-F 3 "" H 1000 4500 50  0001 C CNN
-	1    1000 4500
+P 1000 5000
+F 0 "#PWR0112" H 1000 4750 50  0001 C CNN
+F 1 "GND" V 1005 4872 50  0000 R CNN
+F 2 "" H 1000 5000 50  0001 C CNN
+F 3 "" H 1000 5000 50  0001 C CNN
+	1    1000 5000
 	0    1    1    0
 $EndComp
@@
 L Device:R R33
 U 1 1 5F9F9DE5
-P 1150 4500
-F 0 "R33" V 943 4500 50  0000 C CNN
-F 1 "1k" V 1034 4500 50  0000 C CNN
-F 2 "Resistor_SMD:R_0402_1005Metric" V 1080 4500 50  0001 C CNN
-F 3 "~" H 1150 4500 50  0001 C CNN
-	1    1150 4500
+P 1150 5000
+F 0 "R33" V 943 5000 50  0000 C CNN
+F 1 "1k" V 1034 5000 50  0000 C CNN
+F 2 "Resistor_SMD:R_0402_1005Metric" V 1080 5000 50  0001 C CNN
+F 3 "~" H 1150 5000 50  0001 C CNN
+	1    1150 5000
 	0    1    1    0
 $EndComp
@@
 L Device:R R34
 U 1 1 5F9FA379
-P 1450 4500
-F 0 "R34" V 1243 4500 50  0000 C CNN
-F 1 "10k" V 1334 4500 50  0000 C CNN
-F 2 "Resistor_SMD:R_0402_1005Metric" V 1380 4500 50  0001 C CNN
-F 3 "~" H 1450 4500 50  0001 C CNN
-	1    1450 4500
+P 1450 5000
+F 0 "R34" V 1243 5000 50  0000 C CNN
+F 1 "10k" V 1334 5000 50  0000 C CNN
+F 2 "Resistor_SMD:R_0402_1005Metric" V 1380 5000 50  0001 C CNN
+F 3 "~" H 1450 5000 50  0001 C CNN
+	1    1450 5000
 	0    1    1    0
 $EndComp
 Text Label 1900 4000 0    50   ~ 0
 VI
-Text Label 1600 4500 0    50   ~ 0
+Text Label 1600 5000 0    50   ~ 0
 VBAT
 $Comp
@@
 L Device:R R35
 U 1 1 5F9FC56A
-P 1450 4650
-F 0 "R35" V 1550 4650 50  0000 C CNN
-F 1 "0" V 1650 4650 50  0000 C CNN
-F 2 "Resistor_SMD:R_0402_1005Metric" V 1380 4650 50  0001 C CNN
-F 3 "~" H 1450 4650 50  0001 C CNN
-	1    1450 4650
+P 1450 5150
+F 0 "R35" V 1550 5150 50  0000 C CNN
+F 1 "0" V 1650 5150 50  0000 C CNN
+F 2 "Resistor_SMD:R_0402_1005Metric" V 1380 5150 50  0001 C CNN
+F 3 "~" H 1450 5150 50  0001 C CNN
+	1    1450 5150
 	0    1    1    0
 $EndComp
@@
 Connection ~ 1300 4000
 Wire Wire Line
-	1300 4650 1300 4500
-Connection ~ 1300 4500
+	1300 5150 1300 5000
+Connection ~ 1300 5000
 Text Label 1900 4150 0    50   ~ 0
 IO9
-Text Label 1600 4650 0    50   ~ 0
+Text Label 1600 5150 0    50   ~ 0
 IO10
 Text Label 8600 5000 2    50   ~ 0
@@
 Text Label 8600 4300 2    50   ~ 0
 3V3
+$Comp
+L power:GND #PWR?
+U 1 1 5F9EF8BB
+P 1000 6000
+F 0 "#PWR?" H 1000 5750 50  0001 C CNN
+F 1 "GND" V 1005 5872 50  0000 R CNN
+F 2 "" H 1000 6000 50  0001 C CNN
+F 3 "" H 1000 6000 50  0001 C CNN
+	1    1000 6000
+	0    1    1    0
+$EndComp
+$Comp
+L Device:R R50
+U 1 1 5F9EFE28
+P 1150 6000
+F 0 "R50" V 943 6000 50  0000 C CNN
+F 1 "1k" V 1034 6000 50  0000 C CNN
+F 2 "" V 1080 6000 50  0001 C CNN
+F 3 "~" H 1150 6000 50  0001 C CNN
+	1    1150 6000
+	0    1    1    0
+$EndComp
+$Comp
+L Device:R R51
+U 1 1 5F9F0416
+P 1450 6000
+F 0 "R51" V 1243 6000 50  0000 C CNN
+F 1 "1k" V 1334 6000 50  0000 C CNN
+F 2 "" V 1380 6000 50  0001 C CNN
+F 3 "~" H 1450 6000 50  0001 C CNN
+	1    1450 6000
+	0    1    1    0
+$EndComp
+$Comp
+L Device:R R52
+U 1 1 5F9F0A35
+P 1750 6000
+F 0 "R52" V 1543 6000 50  0000 C CNN
+F 1 "1k" V 1634 6000 50  0000 C CNN
+F 2 "" V 1680 6000 50  0001 C CNN
+F 3 "~" H 1750 6000 50  0001 C CNN
+	1    1750 6000
+	0    1    1    0
+$EndComp
+$Comp
+L Device:R R53
+U 1 1 5F9F1277
+P 1750 6150
+F 0 "R53" V 1850 6150 50  0000 C CNN
+F 1 "0" V 1950 6150 50  0000 C CNN
+F 2 "" V 1680 6150 50  0001 C CNN
+F 3 "~" H 1750 6150 50  0001 C CNN
+	1    1750 6150
+	0    1    1    0
+$EndComp
+Wire Wire Line
+	1600 6150 1300 6150
+Wire Wire Line
+	1300 6150 1300 6000
+Connection ~ 1300 6000
+Text Label 1900 6000 0    50   ~ 0
+VBUS
+Text Label 1900 6150 0    50   ~ 0
+IO12
+Text Label 7300 3900 2    50   ~ 0
+VBUS
+Wire Wire Line
+	6800 4100 7300 4100
+Connection ~ 6800 4100
+Wire Wire Line
+	6800 4200 7300 4200
+Connection ~ 6800 4200
 $EndSCHEMATC

Commit message: doc/kicad: FM01-ES2-1  update README.md
Parts:
- C1: footprint Capacitor_SMD:C_0402_1005Metric -> Capacitor_SMD:C_1206_3216Metric
- R50, R51, R52, R53: footprint (none) -> Resistor_SMD:R_0402_1005Metric
Changed lines of the file:
@@
 F 0 "C1" H 1115 1396 50  0000 L CNN
 F 1 "22u" H 1115 1305 50  0000 L CNN
-F 2 "Capacitor_SMD:C_0402_1005Metric" H 1038 1200 50  0001 C CNN
+F 2 "Capacitor_SMD:C_1206_3216Metric" H 1038 1200 50  0001 C CNN
 F 3 "~" H 1000 1350 50  0001 C CNN
 	1    1000 1350
@@
 3V3
 $Comp
-L power:GND #PWR?
+L power:GND #PWR0113
 U 1 1 5F9EF8BB
 P 1000 6000
-F 0 "#PWR?" H 1000 5750 50  0001 C CNN
+F 0 "#PWR0113" H 1000 5750 50  0001 C CNN
 F 1 "GND" V 1005 5872 50  0000 R CNN
 F 2 "" H 1000 6000 50  0001 C CNN
@@
 F 0 "R50" V 943 6000 50  0000 C CNN
 F 1 "1k" V 1034 6000 50  0000 C CNN
-F 2 "" V 1080 6000 50  0001 C CNN
+F 2 "Resistor_SMD:R_0402_1005Metric" V 1080 6000 50  0001 C CNN
 F 3 "~" H 1150 6000 50  0001 C CNN
 	1    1150 6000
@@
 F 0 "R51" V 1243 6000 50  0000 C CNN
 F 1 "1k" V 1334 6000 50  0000 C CNN
-F 2 "" V 1380 6000 50  0001 C CNN
+F 2 "Resistor_SMD:R_0402_1005Metric" V 1380 6000 50  0001 C CNN
 F 3 "~" H 1450 6000 50  0001 C CNN
 	1    1450 6000
@@
 F 0 "R52" V 1543 6000 50  0000 C CNN
 F 1 "1k" V 1634 6000 50  0000 C CNN
-F 2 "" V 1680 6000 50  0001 C CNN
+F 2 "Resistor_SMD:R_0402_1005Metric" V 1680 6000 50  0001 C CNN
 F 3 "~" H 1750 6000 50  0001 C CNN
 	1    1750 6000
@@
 F 0 "R53" V 1850 6150 50  0000 C CNN
 F 1 "0" V 1950 6150 50  0000 C CNN
-F 2 "" V 1680 6150 50  0001 C CNN
+F 2 "Resistor_SMD:R_0402_1005Metric" V 1680 6150 50  0001 C CNN
 F 3 "~" H 1750 6150 50  0001 C CNN
 	1    1750 6150
