File: doc/kicad/fmesc-1-a/FMESC-1-A/FMESC-1-A.sch (KiCad schematic (older format))
At the start: 5 parts

Commit message: doc/kicad: FMESC-1-A v0.3
Parts:
- JT1, JT2, JT3: footprint fmlibf:JS_2P_1.0mm -> fmlibf:JS_2P_1.0mm_F
Changed lines of the file:
@@
 Sheet 1 5
 Title "FMESC-1-A"
-Date "2020-11-10"
-Rev "v0.2"
+Date "2020-11-14"
+Rev "v0.3"
 Comp "sceext"
 Comment1 ""
@@
 F 0 "JT1" H 918 3217 50  0000 C CNN
 F 1 "Conn_01x02" H 918 3126 50  0000 C CNN
-F 2 "fmlibf:JS_2P_1.0mm" H 1000 3000 50  0001 C CNN
+F 2 "fmlibf:JS_2P_1.0mm_F" H 1000 3000 50  0001 C CNN
 F 3 "~" H 1000 3000 50  0001 C CNN
 	1    1000 3000
@@
 F 0 "JT2" H 918 3717 50  0000 C CNN
 F 1 "Conn_01x02" H 918 3626 50  0000 C CNN
-F 2 "fmlibf:JS_2P_1.0mm" H 1000 3500 50  0001 C CNN
+F 2 "fmlibf:JS_2P_1.0mm_F" H 1000 3500 50  0001 C CNN
 F 3 "~" H 1000 3500 50  0001 C CNN
 	1    1000 3500
@@
 F 0 "JT3" H 918 4217 50  0000 C CNN
 F 1 "Conn_01x02" H 918 4126 50  0000 C CNN
-F 2 "fmlibf:JS_2P_1.0mm" H 1000 4000 50  0001 C CNN
+F 2 "fmlibf:JS_2P_1.0mm_F" H 1000 4000 50  0001 C CNN
 F 3 "~" H 1000 4000 50  0001 C CNN
 	1    1000 4000

Commit message: doc/kicad: FMESC-1-A clean and use FMPCBVDL-1
Parts:
- JB0: footprint fmlibf:JS3x13mm -> fmlibf:JS-JB0
- JG0: footprint fmlibf:JS4x16mm -> fmlibf:JS-JG0
- JT1, JT2, JT3: footprint fmlibf:JS_2P_1.0mm_F -> fmlibf:FMPCBVDL-1-S
Changed lines of the file:
@@
 Sheet 1 5
 Title "FMESC-1-A"
-Date "2020-11-14"
+Date "2020-11-29"
 Rev "v0.3"
 Comp "sceext"
@@
 F 0 "JB0" H 2080 1542 50  0000 L CNN
 F 1 "Conn_01x01" H 2080 1451 50  0000 L CNN
-F 2 "fmlibf:JS3x13mm" H 2000 1500 50  0001 C CNN
+F 2 "fmlibf:JS-JB0" H 2000 1500 50  0001 C CNN
 F 3 "~" H 2000 1500 50  0001 C CNN
 	1    2000 1500
@@
 F 0 "JG0" H 2080 2042 50  0000 L CNN
 F 1 "Conn_01x01" H 2080 1951 50  0000 L CNN
-F 2 "fmlibf:JS4x16mm" H 2000 2000 50  0001 C CNN
+F 2 "fmlibf:JS-JG0" H 2000 2000 50  0001 C CNN
 F 3 "~" H 2000 2000 50  0001 C CNN
 	1    2000 2000
@@
 F 0 "JT1" H 918 3217 50  0000 C CNN
 F 1 "Conn_01x02" H 918 3126 50  0000 C CNN
-F 2 "fmlibf:JS_2P_1.0mm_F" H 1000 3000 50  0001 C CNN
+F 2 "fmlibf:FMPCBVDL-1-S" H 1000 3000 50  0001 C CNN
 F 3 "~" H 1000 3000 50  0001 C CNN
 	1    1000 3000
@@
 F 0 "JT2" H 918 3717 50  0000 C CNN
 F 1 "Conn_01x02" H 918 3626 50  0000 C CNN
-F 2 "fmlibf:JS_2P_1.0mm_F" H 1000 3500 50  0001 C CNN
+F 2 "fmlibf:FMPCBVDL-1-S" H 1000 3500 50  0001 C CNN
 F 3 "~" H 1000 3500 50  0001 C CNN
 	1    1000 3500
@@
 F 0 "JT3" H 918 4217 50  0000 C CNN
 F 1 "Conn_01x02" H 918 4126 50  0000 C CNN
-F 2 "fmlibf:JS_2P_1.0mm_F" H 1000 4000 50  0001 C CNN
+F 2 "fmlibf:FMPCBVDL-1-S" H 1000 4000 50  0001 C CNN
 F 3 "~" H 1000 4000 50  0001 C CNN
 	1    1000 4000

Commit message: doc/kicad: FMESC-1-A v0.3 PCB
Connections:
- net GND: now also JT1.1 (Pin_1), JT1.2 (Pin_2)
- no-connect marks 2 -> 0
Changed lines of the file:
@@
 Text Label 1200 4100 0    50   ~ 0
 VB
-NoConn ~ 1200 3000
-NoConn ~ 1200 3100
+Text Label 1200 3000 0    50   ~ 0
+GND
+Text Label 1200 3100 0    50   ~ 0
+GND
 $EndSCHEMATC
