File: doc/kicad/fmesc-1-a/FMESC-1-A/M1.sch (KiCad schematic (older format))
At the start: 21 parts, among them J1 Conn_01x02, J2 Conn_01x02, J3 Conn_01x02, J4 Conn_01x02, J5 Conn_01x02, J6 Conn_01x02, Q1 AON6504, Q2 AON6504, Q3 AON6504, Q4 AON6504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

Commit message: doc/kicad: FMESC-1-A v0.3
Parts:
- J1, J2, J3, J4, J5, J6: footprint fmlibf:JS_2P_1.0mm -> fmlibf:JS_2P_1.0mm_F
Changed lines of the file:
@@
 Sheet 5 5
 Title "FMESC-1-A  M1"
-Date "2020-11-08"
-Rev "v0.1"
+Date "2020-11-14"
+Rev "v0.3"
 Comp "sceext"
 Comment1 ""
@@
 F 0 "J2" H 1418 4725 50  0000 C CNN
 F 1 "Conn_01x02" H 1418 4816 50  0000 C CNN
-F 2 "fmlibf:JS_2P_1.0mm" H 1500 5050 50  0001 C CNN
+F 2 "fmlibf:JS_2P_1.0mm_F" H 1500 5050 50  0001 C CNN
 F 3 "~" H 1500 5050 50  0001 C CNN
 	1    1500 5050
@@
 F 0 "J1" H 1418 5225 50  0000 C CNN
 F 1 "Conn_01x02" H 1418 5316 50  0000 C CNN
-F 2 "fmlibf:JS_2P_1.0mm" H 1500 5550 50  0001 C CNN
+F 2 "fmlibf:JS_2P_1.0mm_F" H 1500 5550 50  0001 C CNN
 F 3 "~" H 1500 5550 50  0001 C CNN
 	1    1500 5550
@@
 F 0 "J4" H 3918 4725 50  0000 C CNN
 F 1 "Conn_01x02" H 3918 4816 50  0000 C CNN
-F 2 "fmlibf:JS_2P_1.0mm" H 4000 5050 50  0001 C CNN
+F 2 "fmlibf:JS_2P_1.0mm_F" H 4000 5050 50  0001 C CNN
 F 3 "~" H 4000 5050 50  0001 C CNN
 	1    4000 5050
@@
 F 0 "J3" H 3918 5225 50  0000 C CNN
 F 1 "Conn_01x02" H 3918 5316 50  0000 C CNN
-F 2 "fmlibf:JS_2P_1.0mm" H 4000 5550 50  0001 C CNN
+F 2 "fmlibf:JS_2P_1.0mm_F" H 4000 5550 50  0001 C CNN
 F 3 "~" H 4000 5550 50  0001 C CNN
 	1    4000 5550
@@
 F 0 "J6" H 6418 4725 50  0000 C CNN
 F 1 "Conn_01x02" H 6418 4816 50  0000 C CNN
-F 2 "fmlibf:JS_2P_1.0mm" H 6500 5050 50  0001 C CNN
+F 2 "fmlibf:JS_2P_1.0mm_F" H 6500 5050 50  0001 C CNN
 F 3 "~" H 6500 5050 50  0001 C CNN
 	1    6500 5050
@@
 F 0 "J5" H 6418 5225 50  0000 C CNN
 F 1 "Conn_01x02" H 6418 5316 50  0000 C CNN
-F 2 "fmlibf:JS_2P_1.0mm" H 6500 5550 50  0001 C CNN
+F 2 "fmlibf:JS_2P_1.0mm_F" H 6500 5550 50  0001 C CNN
 F 3 "~" H 6500 5550 50  0001 C CNN
 	1    6500 5550

Commit message: doc/kicad: FMESC-1-A clean and use FMPCBVDL-1
Parts:
- J1, J2, J3, J4, J5, J6: footprint fmlibf:JS_2P_1.0mm_F -> fmlibf:FMPCBVDL-1-S
- JB1, JB2, JB3: footprint fmlibf:JS3x5mm -> fmlibf:JS-JBx
- JG1, JG2, JG3: footprint fmlibf:JS2x3.5mm -> fmlibf:JS-Jx
- MA1, MB1, MC1: footprint fmlibf:JS3x3.5mm -> fmlibf:JS-Jx
Changed lines of the file:
@@
 F 0 "MA1" H 3080 5292 50  0000 L CNN
 F 1 "Conn_01x01" H 3080 5201 50  0000 L CNN
-F 2 "fmlibf:JS3x3.5mm" H 3000 5250 50  0001 C CNN
+F 2 "fmlibf:JS-Jx" H 3000 5250 50  0001 C CNN
 F 3 "~" H 3000 5250 50  0001 C CNN
 	1    3000 5250
@@
 F 0 "MB1" H 5580 5292 50  0000 L CNN
 F 1 "Conn_01x01" H 5580 5201 50  0000 L CNN
-F 2 "fmlibf:JS3x3.5mm" H 5500 5250 50  0001 C CNN
+F 2 "fmlibf:JS-Jx" H 5500 5250 50  0001 C CNN
 F 3 "~" H 5500 5250 50  0001 C CNN
 	1    5500 5250
@@
 F 0 "MC1" H 8080 5292 50  0000 L CNN
 F 1 "Conn_01x01" H 8080 5201 50  0000 L CNN
-F 2 "fmlibf:JS3x3.5mm" H 8000 5250 50  0001 C CNN
+F 2 "fmlibf:JS-Jx" H 8000 5250 50  0001 C CNN
 F 3 "~" H 8000 5250 50  0001 C CNN
 	1    8000 5250
@@
 F 0 "JB1" H 3080 4642 50  0000 L CNN
 F 1 "Conn_01x01" H 3080 4551 50  0000 L CNN
-F 2 "fmlibf:JS3x5mm" H 3000 4600 50  0001 C CNN
+F 2 "fmlibf:JS-JBx" H 3000 4600 50  0001 C CNN
 F 3 "~" H 3000 4600 50  0001 C CNN
 	1    3000 4600
@@
 F 0 "JG1" H 3080 5942 50  0000 L CNN
 F 1 "Conn_01x01" H 3080 5851 50  0000 L CNN
-F 2 "fmlibf:JS2x3.5mm" H 3000 5900 50  0001 C CNN
+F 2 "fmlibf:JS-Jx" H 3000 5900 50  0001 C CNN
 F 3 "~" H 3000 5900 50  0001 C CNN
 	1    3000 5900
@@
 F 0 "JB2" H 5580 4642 50  0000 L CNN
 F 1 "Conn_01x01" H 5580 4551 50  0000 L CNN
-F 2 "fmlibf:JS3x5mm" H 5500 4600 50  0001 C CNN
+F 2 "fmlibf:JS-JBx" H 5500 4600 50  0001 C CNN
 F 3 "~" H 5500 4600 50  0001 C CNN
 	1    5500 4600
@@
 F 0 "JB3" H 8080 4642 50  0000 L CNN
 F 1 "Conn_01x01" H 8080 4551 50  0000 L CNN
-F 2 "fmlibf:JS3x5mm" H 8000 4600 50  0001 C CNN
+F 2 "fmlibf:JS-JBx" H 8000 4600 50  0001 C CNN
 F 3 "~" H 8000 4600 50  0001 C CNN
 	1    8000 4600
@@
 F 0 "JG2" H 5580 5942 50  0000 L CNN
 F 1 "Conn_01x01" H 5580 5851 50  0000 L CNN
-F 2 "fmlibf:JS2x3.5mm" H 5500 5900 50  0001 C CNN
+F 2 "fmlibf:JS-Jx" H 5500 5900 50  0001 C CNN
 F 3 "~" H 5500 5900 50  0001 C CNN
 	1    5500 5900
@@
 F 0 "JG3" H 8080 5942 50  0000 L CNN
 F 1 "Conn_01x01" H 8080 5851 50  0000 L CNN
-F 2 "fmlibf:JS2x3.5mm" H 8000 5900 50  0001 C CNN
+F 2 "fmlibf:JS-Jx" H 8000 5900 50  0001 C CNN
 F 3 "~" H 8000 5900 50  0001 C CNN
 	1    8000 5900
@@
 F 0 "J2" H 1418 4725 50  0000 C CNN
 F 1 "Conn_01x02" H 1418 4816 50  0000 C CNN
-F 2 "fmlibf:JS_2P_1.0mm_F" H 1500 5050 50  0001 C CNN
+F 2 "fmlibf:FMPCBVDL-1-S" H 1500 5050 50  0001 C CNN
 F 3 "~" H 1500 5050 50  0001 C CNN
 	1    1500 5050
@@
 F 0 "J1" H 1418 5225 50  0000 C CNN
 F 1 "Conn_01x02" H 1418 5316 50  0000 C CNN
-F 2 "fmlibf:JS_2P_1.0mm_F" H 1500 5550 50  0001 C CNN
+F 2 "fmlibf:FMPCBVDL-1-S" H 1500 5550 50  0001 C CNN
 F 3 "~" H 1500 5550 50  0001 C CNN
 	1    1500 5550
@@
 F 0 "J4" H 3918 4725 50  0000 C CNN
 F 1 "Conn_01x02" H 3918 4816 50  0000 C CNN
-F 2 "fmlibf:JS_2P_1.0mm_F" H 4000 5050 50  0001 C CNN
+F 2 "fmlibf:FMPCBVDL-1-S" H 4000 5050 50  0001 C CNN
 F 3 "~" H 4000 5050 50  0001 C CNN
 	1    4000 5050
@@
 F 0 "J3" H 3918 5225 50  0000 C CNN
 F 1 "Conn_01x02" H 3918 5316 50  0000 C CNN
-F 2 "fmlibf:JS_2P_1.0mm_F" H 4000 5550 50  0001 C CNN
+F 2 "fmlibf:FMPCBVDL-1-S" H 4000 5550 50  0001 C CNN
 F 3 "~" H 4000 5550 50  0001 C CNN
 	1    4000 5550
@@
 F 0 "J6" H 6418 4725 50  0000 C CNN
 F 1 "Conn_01x02" H 6418 4816 50  0000 C CNN
-F 2 "fmlibf:JS_2P_1.0mm_F" H 6500 5050 50  0001 C CNN
+F 2 "fmlibf:FMPCBVDL-1-S" H 6500 5050 50  0001 C CNN
 F 3 "~" H 6500 5050 50  0001 C CNN
 	1    6500 5050
@@
 F 0 "J5" H 6418 5225 50  0000 C CNN
 F 1 "Conn_01x02" H 6418 5316 50  0000 C CNN
-F 2 "fmlibf:JS_2P_1.0mm_F" H 6500 5550 50  0001 C CNN
+F 2 "fmlibf:FMPCBVDL-1-S" H 6500 5550 50  0001 C CNN
 F 3 "~" H 6500 5550 50  0001 C CNN
 	1    6500 5550

Commit message: doc/kicad: FMESC-1-A v0.3 PCB
Parts:
- JG1, JG2, JG3: footprint fmlibf:JS-Jx -> fmlibf:JS-JGx
Changed lines of the file:
@@
 $Descr A4 11693 8268
 encoding utf-8
-Sheet 5 5
+Sheet 2 5
 Title "FMESC-1-A  M1"
 Date "2020-11-14"
@@
 AR Path="/5FA3EBFA/5FA18C7A" Ref="#PWR0111"  Part="1"
 AR Path="/5FA3F05C/5FA18C7A" Ref="#PWR0115"  Part="1"
-F 0 "#PWR0103" H 2500 5750 50  0001 C CNN
+F 0 "#PWR0115" H 2500 5750 50  0001 C CNN
 F 1 "GND" H 2505 5827 50  0000 C CNN
 F 2 "" H 2500 6000 50  0001 C CNN
@@
 AR Path="/5FA3EBFA/5FA18E6D" Ref="Q14"  Part="1"
 AR Path="/5FA3F05C/5FA18E6D" Ref="Q20"  Part="1"
-F 0 "Q2" H 2604 5046 50  0000 L CNN
+F 0 "Q20" H 2604 5046 50  0000 L CNN
 F 1 "AON6504" H 2604 4955 50  0000 L CNN
 F 2 "fmlibf:DFN5x6_8L_EP1_P" H 2600 5100 50  0001 C CNN
@@
 AR Path="/5FA3EBFA/5FA1E885" Ref="Q15"  Part="1"
 AR Path="/5FA3F05C/5FA1E885" Ref="Q21"  Part="1"
-F 0 "Q3" H 5104 5546 50  0000 L CNN
+F 0 "Q21" H 5104 5546 50  0000 L CNN
 F 1 "AON6504" H 5104 5455 50  0000 L CNN
 F 2 "fmlibf:DFN5x6_8L_EP1_P" H 5100 5600 50  0001 C CNN
@@
 AR Path="/5FA3EBFA/5FA1E88B" Ref="#PWR0112"  Part="1"
 AR Path="/5FA3F05C/5FA1E88B" Ref="#PWR0116"  Part="1"
-F 0 "#PWR0104" H 5000 5750 50  0001 C CNN
+F 0 "#PWR0116" H 5000 5750 50  0001 C CNN
 F 1 "GND" H 5005 5827 50  0000 C CNN
 F 2 "" H 5000 6000 50  0001 C CNN
@@
 AR Path="/5FA3EBFA/5FA1E892" Ref="Q16"  Part="1"
 AR Path="/5FA3F05C/5FA1E892" Ref="Q22"  Part="1"
-F 0 "Q4" H 5104 5046 50  0000 L CNN
+F 0 "Q22" H 5104 5046 50  0000 L CNN
 F 1 "AON6504" H 5104 4955 50  0000 L CNN
 F 2 "fmlibf:DFN5x6_8L_EP1_P" H 5100 5100 50  0001 C CNN
@@
 AR Path="/5FA3EBFA/5FA23579" Ref="Q17"  Part="1"
 AR Path="/5FA3F05C/5FA23579" Ref="Q23"  Part="1"
-F 0 "Q5" H 7604 5546 50  0000 L CNN
+F 0 "Q23" H 7604 5546 50  0000 L CNN
 F 1 "AON6504" H 7604 5455 50  0000 L CNN
 F 2 "fmlibf:DFN5x6_8L_EP1_P" H 7600 5600 50  0001 C CNN
@@
 AR Path="/5FA3EBFA/5FA2357F" Ref="#PWR0113"  Part="1"
 AR Path="/5FA3F05C/5FA2357F" Ref="#PWR0117"  Part="1"
-F 0 "#PWR0105" H 7500 5750 50  0001 C CNN
+F 0 "#PWR0117" H 7500 5750 50  0001 C CNN
 F 1 "GND" H 7505 5827 50  0000 C CNN
 F 2 "" H 7500 6000 50  0001 C CNN
@@
 AR Path="/5FA3EBFA/5FA23586" Ref="Q18"  Part="1"
 AR Path="/5FA3F05C/5FA23586" Ref="Q24"  Part="1"
-F 0 "Q6" H 7604 5046 50  0000 L CNN
+F 0 "Q24" H 7604 5046 50  0000 L CNN
 F 1 "AON6504" H 7604 4955 50  0000 L CNN
 F 2 "fmlibf:DFN5x6_8L_EP1_P" H 7600 5100 50  0001 C CNN
@@
 AR Path="/5FA3EBFA/5FA44AA6" Ref="MA3"  Part="1"
 AR Path="/5FA3F05C/5FA44AA6" Ref="MA4"  Part="1"
-F 0 "MA1" H 3080 5292 50  0000 L CNN
+F 0 "MA4" H 3080 5292 50  0000 L CNN
 F 1 "Conn_01x01" H 3080 5201 50  0000 L CNN
 F 2 "fmlibf:JS-Jx" H 3000 5250 50  0001 C CNN
@@
 AR Path="/5FA3EBFA/5FA44F40" Ref="MB3"  Part="1"
 AR Path="/5FA3F05C/5FA44F40" Ref="MB4"  Part="1"
-F 0 "MB1" H 5580 5292 50  0000 L CNN
+F 0 "MB4" H 5580 5292 50  0000 L CNN
 F 1 "Conn_01x01" H 5580 5201 50  0000 L CNN
 F 2 "fmlibf:JS-Jx" H 5500 5250 50  0001 C CNN
@@
 AR Path="/5FA3EBFA/5FA4532B" Ref="MC3"  Part="1"
 AR Path="/5FA3F05C/5FA4532B" Ref="MC4"  Part="1"
-F 0 "MC1" H 8080 5292 50  0000 L CNN
+F 0 "MC4" H 8080 5292 50  0000 L CNN
 F 1 "Conn_01x01" H 8080 5201 50  0000 L CNN
 F 2 "fmlibf:JS-Jx" H 8000 5250 50  0001 C CNN
@@
 AR Path="/5FA3EBFA/5FA6301C" Ref="#PWR0125"  Part="1"
 AR Path="/5FA3F05C/5FA6301C" Ref="#PWR0128"  Part="1"
-F 0 "#PWR0119" H 2500 4350 50  0001 C CNN
+F 0 "#PWR0128" H 2500 4350 50  0001 C CNN
 F 1 "+BATT" H 2515 4673 50  0000 C CNN
 F 2 "" H 2500 4500 50  0001 C CNN
@@
 AR Path="/5FA3EBFA/5FA6A42A" Ref="JB7"  Part="1"
 AR Path="/5FA3F05C/5FA6A42A" Ref="JB10"  Part="1"
-F 0 "JB1" H 3080 4642 50  0000 L CNN
+F 0 "JB10" H 3080 4642 50  0000 L CNN
 F 1 "Conn_01x01" H 3080 4551 50  0000 L CNN
 F 2 "fmlibf:JS-JBx" H 3000 4600 50  0001 C CNN
@@
 AR Path="/5FA3EBFA/5FA7366A" Ref="JG7"  Part="1"
 AR Path="/5FA3F05C/5FA7366A" Ref="JG10"  Part="1"
-F 0 "JG1" H 3080 5942 50  0000 L CNN
+F 0 "JG10" H 3080 5942 50  0000 L CNN
 F 1 "Conn_01x01" H 3080 5851 50  0000 L CNN
-F 2 "fmlibf:JS-Jx" H 3000 5900 50  0001 C CNN
+F 2 "fmlibf:JS-JGx" H 3000 5900 50  0001 C CNN
 F 3 "~" H 3000 5900 50  0001 C CNN
 	1    3000 5900
@@
 AR Path="/5FA3EBFA/5FA76D98" Ref="#PWR0126"  Part="1"
 AR Path="/5FA3F05C/5FA76D98" Ref="#PWR0129"  Part="1"
-F 0 "#PWR0120" H 5000 4350 50  0001 C CNN
+F 0 "#PWR0129" H 5000 4350 50  0001 C CNN
 F 1 "+BATT" H 5015 4673 50  0000 C CNN
 F 2 "" H 5000 4500 50  0001 C CNN
@@
 AR Path="/5FA3EBFA/5FA770E9" Ref="#PWR0127"  Part="1"
 AR Path="/5FA3F05C/5FA770E9" Ref="#PWR0130"  Part="1"
-F 0 "#PWR0121" H 7500 4350 50  0001 C CNN
+F 0 "#PWR0130" H 7500 4350 50  0001 C CNN
 F 1 "+BATT" H 7515 4673 50  0000 C CNN
 F 2 "" H 7500 4500 50  0001 C CNN
@@
 AR Path="/5FA3EBFA/5FA7749F" Ref="JB8"  Part="1"
 AR Path="/5FA3F05C/5FA7749F" Ref="JB11"  Part="1"
-F 0 "JB2" H 5580 4642 50  0000 L CNN
+F 0 "JB11" H 5580 4642 50  0000 L CNN
 F 1 "Conn_01x01" H 5580 4551 50  0000 L CNN
 F 2 "fmlibf:JS-JBx" H 5500 4600 50  0001 C CNN
@@
 AR Path="/5FA3EBFA/5FA7789A" Ref="JB9"  Part="1"
 AR Path="/5FA3F05C/5FA7789A" Ref="JB12"  Part="1"
-F 0 "JB3" H 8080 4642 50  0000 L CNN
+F 0 "JB12" H 8080 4642 50  0000 L CNN
 F 1 "Conn_01x01" H 8080 4551 50  0000 L CNN
 F 2 "fmlibf:JS-JBx" H 8000 4600 50  0001 C CNN
@@
 AR Path="/5FA3EBFA/5FA77F11" Ref="JG8"  Part="1"
 AR Path="/5FA3F05C/5FA77F11" Ref="JG11"  Part="1"
-F 0 "JG2" H 5580 5942 50  0000 L CNN
+F 0 "JG11" H 5580 5942 50  0000 L CNN
 F 1 "Conn_01x01" H 5580 5851 50  0000 L CNN
-F 2 "fmlibf:JS-Jx" H 5500 5900 50  0001 C CNN
+F 2 "fmlibf:JS-JGx" H 5500 5900 50  0001 C CNN
 F 3 "~" H 5500 5900 50  0001 C CNN
 	1    5500 5900
@@
 AR Path="/5FA3EBFA/5FA782C1" Ref="JG9"  Part="1"
 AR Path="/5FA3F05C/5FA782C1" Ref="JG12"  Part="1"
-F 0 "JG3" H 8080 5942 50  0000 L CNN
+F 0 "JG12" H 8080 5942 50  0000 L CNN
 F 1 "Conn_01x01" H 8080 5851 50  0000 L CNN
-F 2 "fmlibf:JS-Jx" H 8000 5900 50  0001 C CNN
+F 2 "fmlibf:JS-JGx" H 8000 5900 50  0001 C CNN
 F 3 "~" H 8000 5900 50  0001 C CNN
 	1    8000 5900
@@
 AR Path="/5FA3EBFA/5FA18782" Ref="Q13"  Part="1"
 AR Path="/5FA3F05C/5FA18782" Ref="Q19"  Part="1"
-F 0 "Q1" H 2604 5546 50  0000 L CNN
+F 0 "Q19" H 2604 5546 50  0000 L CNN
 F 1 "AON6504" H 2604 5455 50  0000 L CNN
 F 2 "fmlibf:DFN5x6_8L_EP1_P" H 2600 5600 50  0001 C CNN
@@
 AR Path="/5FA3EBFA/5FA80AC7" Ref="J14"  Part="1"
 AR Path="/5FA3F05C/5FA80AC7" Ref="J20"  Part="1"
-F 0 "J2" H 1418 4725 50  0000 C CNN
+F 0 "J20" H 1418 4725 50  0000 C CNN
 F 1 "Conn_01x02" H 1418 4816 50  0000 C CNN
 F 2 "fmlibf:FMPCBVDL-1-S" H 1500 5050 50  0001 C CNN
@@
 AR Path="/5FA3EBFA/5FA8AB34" Ref="J13"  Part="1"
 AR Path="/5FA3F05C/5FA8AB34" Ref="J19"  Part="1"
-F 0 "J1" H 1418 5225 50  0000 C CNN
+F 0 "J19" H 1418 5225 50  0000 C CNN
 F 1 "Conn_01x02" H 1418 5316 50  0000 C CNN
 F 2 "fmlibf:FMPCBVDL-1-S" H 1500 5550 50  0001 C CNN
@@
 AR Path="/5FA3EBFA/5FA8C1AD" Ref="#PWR0131"  Part="1"
 AR Path="/5FA3F05C/5FA8C1AD" Ref="#PWR0106"  Part="1"
-F 0 "#PWR0139" H 1700 5300 50  0001 C CNN
+F 0 "#PWR0106" H 1700 5300 50  0001 C CNN
 F 1 "GND" H 1705 5377 50  0000 C CNN
 F 2 "" H 1700 5550 50  0001 C CNN
@@
 AR Path="/5FA3EBFA/5FA8E220" Ref="J16"  Part="1"
 AR Path="/5FA3F05C/5FA8E220" Ref="J22"  Part="1"
-F 0 "J4" H 3918 4725 50  0000 C CNN
+F 0 "J22" H 3918 4725 50  0000 C CNN
 F 1 "Conn_01x02" H 3918 4816 50  0000 C CNN
 F 2 "fmlibf:FMPCBVDL-1-S" H 4000 5050 50  0001 C CNN
@@
 AR Path="/5FA3EBFA/5FA8E226" Ref="J15"  Part="1"
 AR Path="/5FA3F05C/5FA8E226" Ref="J21"  Part="1"
-F 0 "J3" H 3918 5225 50  0000 C CNN
+F 0 "J21" H 3918 5225 50  0000 C CNN
 F 1 "Conn_01x02" H 3918 5316 50  0000 C CNN
 F 2 "fmlibf:FMPCBVDL-1-S" H 4000 5550 50  0001 C CNN
@@
 AR Path="/5FA3EBFA/5FA8E22F" Ref="#PWR0132"  Part="1"
 AR Path="/5FA3F05C/5FA8E22F" Ref="#PWR0110"  Part="1"
-F 0 "#PWR0140" H 4200 5300 50  0001 C CNN
+F 0 "#PWR0110" H 4200 5300 50  0001 C CNN
 F 1 "GND" H 4205 5377 50  0000 C CNN
 F 2 "" H 4200 5550 50  0001 C CNN
@@
 AR Path="/5FA3EBFA/5FA8EDC1" Ref="J18"  Part="1"
 AR Path="/5FA3F05C/5FA8EDC1" Ref="J24"  Part="1"
-F 0 "J6" H 6418 4725 50  0000 C CNN
+F 0 "J24" H 6418 4725 50  0000 C CNN
 F 1 "Conn_01x02" H 6418 4816 50  0000 C CNN
 F 2 "fmlibf:FMPCBVDL-1-S" H 6500 5050 50  0001 C CNN
@@
 AR Path="/5FA3EBFA/5FA8EDC7" Ref="J17"  Part="1"
 AR Path="/5FA3F05C/5FA8EDC7" Ref="J23"  Part="1"
-F 0 "J5" H 6418 5225 50  0000 C CNN
+F 0 "J23" H 6418 5225 50  0000 C CNN
 F 1 "Conn_01x02" H 6418 5316 50  0000 C CNN
 F 2 "fmlibf:FMPCBVDL-1-S" H 6500 5550 50  0001 C CNN
@@
 AR Path="/5FA3EBFA/5FA8EDD0" Ref="#PWR0133"  Part="1"
 AR Path="/5FA3F05C/5FA8EDD0" Ref="#PWR0114"  Part="1"
-F 0 "#PWR0141" H 6700 5300 50  0001 C CNN
+F 0 "#PWR0114" H 6700 5300 50  0001 C CNN
 F 1 "GND" H 6705 5377 50  0000 C CNN
 F 2 "" H 6700 5550 50  0001 C CNN
