File: doc/kicad/fm02-b-1/FM02-B-1/FM02-B-1.kicad_pcb (KiCad board)
At the start: 2 copper layers, 0 parts

Commit message: doc/kicad: FM02-B-1 PCB border (edge.cuts)
Other:
- board outline added: 100 x 100 mm
