File: doc/kicad/fmpcbvdl-1/FMPCBVDL-1/FMPCBVDL-1.kicad_pcb (KiCad board)
At the start: 2 copper layers, 0 parts

Commit message: doc/kicad: FMPCBVDL-1 v0.1
Parts:
- added J1: Conn_01x02, fmlibf:FMPCBVDL-1-H, F.Cu at (38.0, 41.0)
- added J2: Conn_01x02, fmlibf:FMPCBVDL-1-H, F.Cu at (43.0, 41.0)
- added J3: Conn_01x02, fmlibf:FMPCBVDL-1-H, F.Cu at (48.0, 41.0)
Other:
- board outline added: 16 x 4 mm
Changed lines of the file:
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@@
   (general
     (thickness 1.6)
-    (drawings 0)
+    (drawings 6)
     (tracks 0)
     (zones 0)
-    (modules 0)
-    (nets 1)
+    (modules 3)
+    (nets 7)
   )
   (page A4)
@@
     (pad_drill 0.762)
     (pad_to_mask_clearance 0)
-    (aux_axis_origin 40.5 89.5)
-    (grid_origin 53 77)
+    (aux_axis_origin 35 43)
+    (grid_origin 43 41)
     (visible_elements FFFDFF7F)
     (pcbplotparams
@@
   )
   (net 0 "")
+  (net 1 "Net-(J1-Pad2)")
+  (net 2 "Net-(J1-Pad1)")
+  (net 3 "Net-(J2-Pad2)")
+  (net 4 "Net-(J2-Pad1)")
+  (net 5 "Net-(J3-Pad2)")
+  (net 6 "Net-(J3-Pad1)")
   (net_class Default "This is the default net class."
     (clearance 0.16)
@@
     (diff_pair_width 0.16)
     (diff_pair_gap 0.16)
-  )
+    (add_net "Net-(J1-Pad1)")
+    (add_net "Net-(J1-Pad2)")
+    (add_net "Net-(J2-Pad1)")
+    (add_net "Net-(J2-Pad2)")
+    (add_net "Net-(J3-Pad1)")
+    (add_net "Net-(J3-Pad2)")
+  )
+  (module fmlibf:FMPCBVDL-1-H (layer F.Cu)
+    (at 48 41)
+    (fp_text reference J3 (at 0 1.8) (layer F.SilkS) hide
+      (effects (font (size 1 1) (thickness 0.15)))
+    )
+    (fp_text value Conn_01x02 (at 0 -1.7) (layer F.Fab)
+      (effects (font (size 1 1) (thickness 0.15)))
+    )
+    (fp_line (start -1.4 -0.7) (end 1.4 -0.7) (layer Cmts.User) (width 0.12))
+    (fp_line (start 1.4 -0.7) (end 1.4 0.7) (layer Cmts.User) (width 0.12))
+    (fp_line (start 1.4 0.7) (end -1.4 0.7) (layer Cmts.User) (width 0.12))
+    (fp_line (start -1.4 0.7) (end -1.4 -0.7) (layer Cmts.User) (width 0.12))
+    (fp_line (start -1.5 -0.8) (end 1.5 -0.8) (layer F.SilkS) (width 0.2))
+    (fp_line (start 1.5 0.8) (end -1.5 0.8) (layer F.SilkS) (width 0.2))
+    (fp_line (start -1.5 -0.8) (end 1.5 -0.8) (layer B.SilkS) (width 0.2))
+    (fp_line (start -1.5 0.8) (end 1.5 0.8) (layer B.SilkS) (width 0.2))
+    (pad 2 thru_hole rect (at 0.8 0) (size 1.2 1.4) (drill 0.9) (layers *.Cu *.Mask)
+      (net 5 "Net-(J3-Pad2)"))
+    (pad 1 thru_hole rect (at -0.8 0) (size 1.2 1.4) (drill 0.9) (layers *.Cu *.Mask)
+      (net 6 "Net-(J3-Pad1)"))
+  )
+  (module fmlibf:FMPCBVDL-1-H (layer F.Cu)
+    (at 43 41)
+    (fp_text reference J2 (at 0 1.8) (layer F.SilkS) hide
+      (effects (font (size 1 1) (thickness 0.15)))
+    )
+    (fp_text value Conn_01x02 (at 0 -1.7) (layer F.Fab)
+      (effects (font (size 1 1) (thickness 0.15)))
+    )
+    (fp_line (start -1.4 -0.7) (end 1.4 -0.7) (layer Cmts.User) (width 0.12))
+    (fp_line (start 1.4 -0.7) (end 1.4 0.7) (layer Cmts.User) (width 0.12))
+    (fp_line (start 1.4 0.7) (end -1.4 0.7) (layer Cmts.User) (width 0.12))
+    (fp_line (start -1.4 0.7) (end -1.4 -0.7) (layer Cmts.User) (width 0.12))
+    (fp_line (start -1.5 -0.8) (end 1.5 -0.8) (layer F.SilkS) (width 0.2))
+    (fp_line (start 1.5 0.8) (end -1.5 0.8) (layer F.SilkS) (width 0.2))
+    (fp_line (start -1.5 -0.8) (end 1.5 -0.8) (layer B.SilkS) (width 0.2))
+    (fp_line (start -1.5 0.8) (end 1.5 0.8) (layer B.SilkS) (width 0.2))
+    (pad 2 thru_hole rect (at 0.8 0) (size 1.2 1.4) (drill 0.9) (layers *.Cu *.Mask)
+      (net 3 "Net-(J2-Pad2)"))
+    (pad 1 thru_hole rect (at -0.8 0) (size 1.2 1.4) (drill 0.9) (layers *.Cu *.Mask)
+      (net 4 "Net-(J2-Pad1)"))
+  )
+  (module fmlibf:FMPCBVDL-1-H (layer F.Cu)
+    (at 38 41)
+    (fp_text reference J1 (at 0 1.8) (layer F.SilkS) hide
+      (effects (font (size 1 1) (thickness 0.15)))
+    )
+    (fp_text value Conn_01x02 (at 0 -1.7) (layer F.Fab)
+      (effects (font (size 1 1) (thickness 0.15)))
+    )
+    (fp_line (start -1.4 -0.7) (end 1.4 -0.7) (layer Cmts.User) (width 0.12))
+    (fp_line (start 1.4 -0.7) (end 1.4 0.7) (layer Cmts.User) (width 0.12))
+    (fp_line (start 1.4 0.7) (end -1.4 0.7) (layer Cmts.User) (width 0.12))
+    (fp_line (start -1.4 0.7) (end -1.4 -0.7) (layer Cmts.User) (width 0.12))
+    (fp_line (start -1.5 -0.8) (end 1.5 -0.8) (layer F.SilkS) (width 0.2))
+    (fp_line (start 1.5 0.8) (end -1.5 0.8) (layer F.SilkS) (width 0.2))
+    (fp_line (start -1.5 -0.8) (end 1.5 -0.8) (layer B.SilkS) (width 0.2))
+    (fp_line (start -1.5 0.8) (end 1.5 0.8) (layer B.SilkS) (width 0.2))
+    (pad 2 thru_hole rect (at 0.8 0) (size 1.2 1.4) (drill 0.9) (layers *.Cu *.Mask)
+      (net 1 "Net-(J1-Pad2)"))
+    (pad 1 thru_hole rect (at -0.8 0) (size 1.2 1.4) (drill 0.9) (layers *.Cu *.Mask)
+      (net 2 "Net-(J1-Pad1)"))
+  )
+  (dimension 4 (width 0.16) (layer Cmts.User)
+    (gr_text "4.000 mm" (at 31.72 41 270) (layer Cmts.User)
+      (effects (font (size 1 0.5) (thickness 0.12)))
+    )
+    (feature1 (pts (xy 35 43) (xy 32.413579 43)))
+    (feature2 (pts (xy 35 39) (xy 32.413579 39)))
+    (crossbar (pts (xy 33 39) (xy 33 43)))
+    (arrow1a (pts (xy 33 43) (xy 32.413579 41.873496)))
+    (arrow1b (pts (xy 33 43) (xy 33.586421 41.873496)))
+    (arrow2a (pts (xy 33 39) (xy 32.413579 40.126504)))
+    (arrow2b (pts (xy 33 39) (xy 33.586421 40.126504)))
+  )
+  (dimension 16 (width 0.16) (layer Cmts.User)
+    (gr_text "16.000 mm" (at 43 35.72) (layer Cmts.User)
+      (effects (font (size 1 0.5) (thickness 0.12)))
+    )
+    (feature1 (pts (xy 51 39) (xy 51 36.413579)))
+    (feature2 (pts (xy 35 39) (xy 35 36.413579)))
+    (crossbar (pts (xy 35 37) (xy 51 37)))
+    (arrow1a (pts (xy 51 37) (xy 49.873496 37.586421)))
+    (arrow1b (pts (xy 51 37) (xy 49.873496 36.413579)))
+    (arrow2a (pts (xy 35 37) (xy 36.126504 37.586421)))
+    (arrow2b (pts (xy 35 37) (xy 36.126504 36.413579)))
+  )
+  (gr_line (start 35 43) (end 35 39) (layer Edge.Cuts) (width 0.2))
+  (gr_line (start 51 43) (end 35 43) (layer Edge.Cuts) (width 0.2))
+  (gr_line (start 51 39) (end 51 43) (layer Edge.Cuts) (width 0.2))
+  (gr_line (start 35 39) (end 51 39) (layer Edge.Cuts) (width 0.2))
 )
