File: doc/kicad/fmpcbvdl-1/FMPCBVDL-1/FMPCBVDL-1.sch (KiCad schematic (older format))
At the start: 3 parts, among them J1 Conn_01x02, J2 Conn_01x02, J3 Conn_01x02

Commit message: doc/kicad: FMPCBVDL-1 v0.1
Parts:
- J1, J2, J3: footprint (none) -> fmlibf:FMPCBVDL-1-H
Changed lines of the file:
@@
 F 0 "J2" H 2030 1942 50  0000 L CNN
 F 1 "Conn_01x02" H 2030 1851 50  0000 L CNN
-F 2 "" H 1950 1950 50  0001 C CNN
+F 2 "fmlibf:FMPCBVDL-1-H" H 1950 1950 50  0001 C CNN
 F 3 "~" H 1950 1950 50  0001 C CNN
 	1    1950 1950
@@
 F 0 "J3" H 2030 2442 50  0000 L CNN
 F 1 "Conn_01x02" H 2030 2351 50  0000 L CNN
-F 2 "" H 1950 2450 50  0001 C CNN
+F 2 "fmlibf:FMPCBVDL-1-H" H 1950 2450 50  0001 C CNN
 F 3 "~" H 1950 2450 50  0001 C CNN
 	1    1950 2450
@@
 F 0 "J1" H 2030 1442 50  0000 L CNN
 F 1 "Conn_01x02" H 2030 1351 50  0000 L CNN
-F 2 "" H 1950 1450 50  0001 C CNN
+F 2 "fmlibf:FMPCBVDL-1-H" H 1950 1450 50  0001 C CNN
 F 3 "~" H 1950 1450 50  0001 C CNN
 	1    1950 1450
