File: doc/kicad/fmsmd-2/FMSMD-2/FMSMD-2.kicad_pcb (KiCad board)
At the start: 2 copper layers, 0 parts

Commit message: doc/kicad: FMSMD-2 PCB v0.1 (1-way)
Parts:
- added C10: 10u, Capacitor_SMD:C_0805_2012Metric, B.Cu at (47.6, 90.5)
- added C11: 10n, Capacitor_SMD:C_0402_1005Metric, B.Cu at (49.4, 89.5)
- added C12: 2.2u, Capacitor_SMD:C_0402_1005Metric, B.Cu at (49.4, 91.5)
- added JAO11: Conn_01x01, fmlibf:JS-1x2mm, F.Cu at (56.8, 92.5)
- added JAO12: Conn_01x01, fmlibf:JS-1x2mm, F.Cu at (56.8, 91.2)
- added JBO11: Conn_01x01, fmlibf:JS-1x2mm, F.Cu at (56.8, 88.5)
- added JBO12: Conn_01x01, fmlibf:JS-1x2mm, F.Cu at (56.8, 89.8)
- added JC1: Conn_01x12, fmlibf:JS_12P_1.0mm, F.Cu at (44.5, 90.5)
- added JG1: Conn_01x01, fmlibf:JS-1x2mm, F.Cu at (47.0, 91.2)
- added JQD1: Conn_01x01, fmlibf:JS-Jx, B.Cu at (58.5, 86.5)
- added JQG1: Conn_01x01, fmlibf:JS-1x1mm, B.Cu at (61.5, 86.5)
- added JQS1: Conn_01x01, fmlibf:JS-JBx, B.Cu at (59.5, 94.5)
- added JVM1: Conn_01x01, fmlibf:JS-1x2mm, F.Cu at (47.0, 89.8)
- added Q1: AON6504, fmlibf:DFN5x6_8L_EP1_P, B.Cu at (59.5, 90.5)
- added Q11: AO3422, Package_TO_SOT_SMD:SOT-23, F.Cu at (53.5, 95.0)
- added Q12: AO3422, Package_TO_SOT_SMD:SOT-23, B.Cu at (51.7, 86.2)
- added R11: 0, Resistor_SMD:R_0603_1608Metric, B.Cu at (53.5, 92.0)
- added R12: 0, Resistor_SMD:R_0603_1608Metric, B.Cu at (53.5, 89.0)
- added R13: 0, Resistor_SMD:R_0603_1608Metric, B.Cu at (53.5, 93.0)
- added R14: 0, Resistor_SMD:R_0603_1608Metric, B.Cu at (53.5, 88.0)
- added R15: 0, Resistor_SMD:R_0402_1005Metric, B.Cu at (54.4, 93.7)
- added R16: 0, Resistor_SMD:R_0402_1005Metric, B.Cu at (54.4, 87.3)
- added R18: 10k, Resistor_SMD:R_0402_1005Metric, F.Cu at (48.0, 86.5)
- added U1: HR8833MTE, fmlibf:HTSSOP-16-1EP_4.4x5mm_P0.65mm_EP3x3mm, F.Cu at (52.0, 90.5)
Routing:
- net GND: track 0.00 -> 21.3 mm, vias 0 -> 6
- net /M1/VIS: track 0.00 -> 20.6 mm, vias 0 -> 1
- net /M1/NFAULT: track 0.00 -> 10.9 mm
- net /M1/NSLEEP: track 0.00 -> 10.7 mm
- net /M1/B2: track 0.00 -> 4.87 mm
- net /M1/A2: track 0.00 -> 4.87 mm
- net /M1/B1: track 0.00 -> 4.73 mm
- net /M1/A1: track 0.00 -> 4.73 mm
- net /M1/3V3: track 0.00 -> 3.49 mm
- net /M1/VM: track 0.00 -> 2.90 mm, vias 0 -> 1
- net /M1/BIS: track 0.00 -> 2.52 mm, vias 0 -> 1
- net /M1/AIS: track 0.00 -> 2.52 mm, vias 0 -> 1
- net Net-(Q12-Pad1): track 0.00 -> 2.32 mm
- net /M1/BO2: track 0.00 -> 1.68 mm
- net /M1/AO2: track 0.00 -> 1.68 mm
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- added copper zone on B.Cu, net GND
- added copper zone on F.Cu, net GND
Other:
- board outline added: 20 x 50 mm
- board text added: "+"
- board text added: "2020-12-04"
- board text added: "A"
- board text added: "B"
- board text added: "FMSMD-2 v0.1"

Commit message: doc/kicad: FMSMD-2 v0.1 PCB
Parts:
- added C20: 10u, Capacitor_SMD:C_0805_2012Metric, B.Cu at (47.6, 78.5)
- added C21: 10n, Capacitor_SMD:C_0402_1005Metric, B.Cu at (49.4, 77.5)
- added C22: 2.2u, Capacitor_SMD:C_0402_1005Metric, B.Cu at (49.4, 79.5)
- added C30: 10u, Capacitor_SMD:C_0805_2012Metric, B.Cu at (47.6, 65.5)
- added C31: 10n, Capacitor_SMD:C_0402_1005Metric, B.Cu at (49.4, 64.5)
- added C32: 2.2u, Capacitor_SMD:C_0402_1005Metric, B.Cu at (49.4, 66.5)
- added C40: 10u, Capacitor_SMD:C_0805_2012Metric, B.Cu at (47.6, 53.5)
- added C41: 10n, Capacitor_SMD:C_0402_1005Metric, B.Cu at (49.4, 52.5)
- added C42: 2.2u, Capacitor_SMD:C_0402_1005Metric, B.Cu at (49.4, 54.5)
- added JAO21: Conn_01x01, fmlibf:JS-1x2mm, F.Cu at (56.8, 80.5)
- added JAO22: Conn_01x01, fmlibf:JS-1x2mm, F.Cu at (56.8, 79.2)
- added JAO31: Conn_01x01, fmlibf:JS-1x2mm, F.Cu at (56.8, 67.5)
- added JAO32: Conn_01x01, fmlibf:JS-1x2mm, F.Cu at (56.8, 66.2)
- added JAO41: Conn_01x01, fmlibf:JS-1x2mm, F.Cu at (56.8, 55.5)
- added JAO42: Conn_01x01, fmlibf:JS-1x2mm, F.Cu at (56.8, 54.2)
- added JBO21: Conn_01x01, fmlibf:JS-1x2mm, F.Cu at (56.8, 76.5)
- added JBO22: Conn_01x01, fmlibf:JS-1x2mm, F.Cu at (56.8, 77.8)
- added JBO31: Conn_01x01, fmlibf:JS-1x2mm, F.Cu at (56.8, 63.5)
- added JBO32: Conn_01x01, fmlibf:JS-1x2mm, F.Cu at (56.8, 64.8)
- added JBO41: Conn_01x01, fmlibf:JS-1x2mm, F.Cu at (56.8, 51.5)
- added JBO42: Conn_01x01, fmlibf:JS-1x2mm, F.Cu at (56.8, 52.8)
- added JC2: Conn_01x12, fmlibf:JS_12P_1.0mm, F.Cu at (44.5, 78.5)
- added JC3: Conn_01x12, fmlibf:JS_12P_1.0mm, F.Cu at (44.5, 65.5)
- added JC4: Conn_01x12, fmlibf:JS_12P_1.0mm, F.Cu at (44.5, 53.5)
- added JG2: Conn_01x01, fmlibf:JS-1x2mm, F.Cu at (47.0, 79.2)
- added JG3: Conn_01x01, fmlibf:JS-1x2mm, F.Cu at (47.0, 66.2)
- added JG4: Conn_01x01, fmlibf:JS-1x2mm, F.Cu at (47.0, 54.2)
- added JQD2: Conn_01x01, fmlibf:JS-Jx, B.Cu at (58.5, 74.5)
- added JQD3: Conn_01x01, fmlibf:JS-Jx, B.Cu at (58.5, 61.5)
- added JQD4: Conn_01x01, fmlibf:JS-Jx, B.Cu at (58.5, 49.5)
- added JQG2: Conn_01x01, fmlibf:JS-1x1mm, B.Cu at (61.5, 74.5)
- added JQG3: Conn_01x01, fmlibf:JS-1x1mm, B.Cu at (61.5, 61.5)
- added JQG4: Conn_01x01, fmlibf:JS-1x1mm, B.Cu at (61.5, 49.5)
- added JQS2: Conn_01x01, fmlibf:JS-JBx, B.Cu at (59.5, 82.5)
- added JQS3: Conn_01x01, fmlibf:JS-JBx, B.Cu at (59.5, 69.5)
- added JQS4: Conn_01x01, fmlibf:JS-JBx, B.Cu at (59.5, 57.5)
- added JVM2: Conn_01x01, fmlibf:JS-1x2mm, F.Cu at (47.0, 77.8)
- added JVM3: Conn_01x01, fmlibf:JS-1x2mm, F.Cu at (47.0, 64.8)
- added JVM4: Conn_01x01, fmlibf:JS-1x2mm, F.Cu at (47.0, 52.8)
- added Q2: AON6504, fmlibf:DFN5x6_8L_EP1_P, B.Cu at (59.5, 78.5)
- added Q21: AO3422, Package_TO_SOT_SMD:SOT-23, F.Cu at (53.5, 83.0)
- added Q22: AO3422, Package_TO_SOT_SMD:SOT-23, B.Cu at (51.7, 74.2)
- added Q3: AON6504, fmlibf:DFN5x6_8L_EP1_P, B.Cu at (59.5, 65.5)
- added Q31: AO3422, Package_TO_SOT_SMD:SOT-23, F.Cu at (53.5, 70.0)
- added Q32: AO3422, Package_TO_SOT_SMD:SOT-23, B.Cu at (51.7, 61.2)
- added Q4: AON6504, fmlibf:DFN5x6_8L_EP1_P, B.Cu at (59.5, 53.5)
- added Q41: AO3422, Package_TO_SOT_SMD:SOT-23, F.Cu at (53.5, 58.0)
- added Q42: AO3422, Package_TO_SOT_SMD:SOT-23, B.Cu at (51.7, 49.2)
- added R21: 0, Resistor_SMD:R_0603_1608Metric, B.Cu at (53.5, 80.0)
- added R22: 0, Resistor_SMD:R_0603_1608Metric, B.Cu at (53.5, 77.0)
- added R23: 0, Resistor_SMD:R_0603_1608Metric, B.Cu at (53.5, 81.0)
- added R24: 0, Resistor_SMD:R_0603_1608Metric, B.Cu at (53.5, 76.0)
- added R25: 0, Resistor_SMD:R_0402_1005Metric, B.Cu at (54.4, 81.7)
- added R26: 0, Resistor_SMD:R_0402_1005Metric, B.Cu at (54.4, 75.3)
- added R28: 10k, Resistor_SMD:R_0402_1005Metric, F.Cu at (48.0, 74.5)
- added R31: 0, Resistor_SMD:R_0603_1608Metric, B.Cu at (53.5, 67.0)
- added R32: 0, Resistor_SMD:R_0603_1608Metric, B.Cu at (53.5, 64.0)
- added R33: 0, Resistor_SMD:R_0603_1608Metric, B.Cu at (53.5, 68.0)
- added R34: 0, Resistor_SMD:R_0603_1608Metric, B.Cu at (53.5, 63.0)
- added R35: 0, Resistor_SMD:R_0402_1005Metric, B.Cu at (54.4, 68.7)
- added R36: 0, Resistor_SMD:R_0402_1005Metric, B.Cu at (54.4, 62.3)
- added R38: 10k, Resistor_SMD:R_0402_1005Metric, F.Cu at (48.0, 61.5)
- added R41: 0, Resistor_SMD:R_0603_1608Metric, B.Cu at (53.5, 55.0)
- added R42: 0, Resistor_SMD:R_0603_1608Metric, B.Cu at (53.5, 52.0)
- added R43: 0, Resistor_SMD:R_0603_1608Metric, B.Cu at (53.5, 56.0)
- added R44: 0, Resistor_SMD:R_0603_1608Metric, B.Cu at (53.5, 51.0)
- added R45: 0, Resistor_SMD:R_0402_1005Metric, B.Cu at (54.4, 56.7)
- added R46: 0, Resistor_SMD:R_0402_1005Metric, B.Cu at (54.4, 50.3)
- added R48: 10k, Resistor_SMD:R_0402_1005Metric, F.Cu at (48.0, 49.5)
- added U2: HR8833MTE, fmlibf:HTSSOP-16-1EP_4.4x5mm_P0.65mm_EP3x3mm, F.Cu at (52.0, 78.5)
- added U3: HR8833MTE, fmlibf:HTSSOP-16-1EP_4.4x5mm_P0.65mm_EP3x3mm, F.Cu at (52.0, 65.5)
- added U4: HR8833MTE, fmlibf:HTSSOP-16-1EP_4.4x5mm_P0.65mm_EP3x3mm, F.Cu at (52.0, 53.5)
Routing:
- net GND: track 21.3 -> 85.3 mm, vias 6 -> 24
- net /M4/VIS: track 0.00 -> 20.6 mm, vias 0 -> 1
- net /M3/VIS: track 0.00 -> 20.6 mm, vias 0 -> 1
- net /M2/VIS: track 0.00 -> 20.6 mm, vias 0 -> 1
- net /M4/NFAULT: track 0.00 -> 10.9 mm
- net /M3/NFAULT: track 0.00 -> 10.9 mm
- net /M2/NFAULT: track 0.00 -> 10.9 mm
- net /M4/NSLEEP: track 0.00 -> 10.7 mm
- net /M3/NSLEEP: track 0.00 -> 10.7 mm
- net /M2/NSLEEP: track 0.00 -> 10.7 mm
- net /M4/B2: track 0.00 -> 4.87 mm
- net /M4/A2: track 0.00 -> 4.87 mm
- net /M3/B2: track 0.00 -> 4.87 mm
- net /M3/A2: track 0.00 -> 4.87 mm
- net /M2/B2: track 0.00 -> 4.87 mm
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