File: doc/kicad/fmsmd-2/FMSMD-2/FMSMD-2.sch (KiCad schematic (older format))
At the start: 0 parts

Commit message: doc/kicad: FMSMD-2 v0.1 PCB
Changed lines of the file:
@@
 $Descr A4 11693 8268
 encoding utf-8
-Sheet 1 2
+Sheet 1 5
 Title "FMSMD-2"
-Date "2020-12-03"
+Date "2020-12-04"
 Rev "v0.1"
 Comp "sceext"
@@
 F1 "M1.sch" 50
 $EndSheet
+$Sheet
+S 7000 1500 1000 1000
+U 5FCA1C8C
+F0 "M2" 50
+F1 "M1.sch" 50
+$EndSheet
+$Sheet
+S 5500 3000 1000 1000
+U 5FCA1CC4
+F0 "M3" 50
+F1 "M1.sch" 50
+$EndSheet
+$Sheet
+S 7000 3000 1000 1000
+U 5FCA1CE0
+F0 "M4" 50
+F1 "M1.sch" 50
+$EndSheet
