File: doc/kicad/fmsmd-2/FMSMD-2/M1.sch (KiCad schematic (older format))
At the start: 24 parts, among them Q1 AON6504, Q11 AO3422, Q12 AO3422, U1 HR8833MTE

Commit message: doc/kicad: FMSMD-2 PCB v0.1 (1-way)
Parts:
- JAO11, JAO12, JBO11, JBO12, JG1, JVM1: footprint fmlibf:JS-1x1mm -> fmlibf:JS-1x2mm
Changed lines of the file:
@@
 Sheet 2 2
 Title "FMSMD-2/M1"
-Date "2020-12-03"
+Date "2020-12-04"
 Rev "v0.1"
 Comp "sceext"
@@
 F 0 "JVM1" H 1418 3275 50  0000 C CNN
 F 1 "Conn_01x01" H 1418 3366 50  0000 C CNN
-F 2 "fmlibf:JS-1x1mm" H 1500 3500 50  0001 C CNN
+F 2 "fmlibf:JS-1x2mm" H 1500 3500 50  0001 C CNN
 F 3 "~" H 1500 3500 50  0001 C CNN
 	1    1500 3500
@@
 F 0 "JG1" H 1418 3775 50  0000 C CNN
 F 1 "Conn_01x01" H 1418 3866 50  0000 C CNN
-F 2 "fmlibf:JS-1x1mm" H 1500 4000 50  0001 C CNN
+F 2 "fmlibf:JS-1x2mm" H 1500 4000 50  0001 C CNN
 F 3 "~" H 1500 4000 50  0001 C CNN
 	1    1500 4000
@@
 F 0 "JAO11" H 1418 4275 50  0000 C CNN
 F 1 "Conn_01x01" H 1418 4366 50  0000 C CNN
-F 2 "fmlibf:JS-1x1mm" H 1500 4500 50  0001 C CNN
+F 2 "fmlibf:JS-1x2mm" H 1500 4500 50  0001 C CNN
 F 3 "~" H 1500 4500 50  0001 C CNN
 	1    1500 4500
@@
 F 0 "JAO12" H 1418 4775 50  0000 C CNN
 F 1 "Conn_01x01" H 1418 4866 50  0000 C CNN
-F 2 "fmlibf:JS-1x1mm" H 1500 5000 50  0001 C CNN
+F 2 "fmlibf:JS-1x2mm" H 1500 5000 50  0001 C CNN
 F 3 "~" H 1500 5000 50  0001 C CNN
 	1    1500 5000
@@
 F 0 "JBO12" H 1418 5275 50  0000 C CNN
 F 1 "Conn_01x01" H 1418 5366 50  0000 C CNN
-F 2 "fmlibf:JS-1x1mm" H 1500 5500 50  0001 C CNN
+F 2 "fmlibf:JS-1x2mm" H 1500 5500 50  0001 C CNN
 F 3 "~" H 1500 5500 50  0001 C CNN
 	1    1500 5500
@@
 F 0 "JBO11" H 1418 5775 50  0000 C CNN
 F 1 "Conn_01x01" H 1418 5866 50  0000 C CNN
-F 2 "fmlibf:JS-1x1mm" H 1500 6000 50  0001 C CNN
+F 2 "fmlibf:JS-1x2mm" H 1500 6000 50  0001 C CNN
 F 3 "~" H 1500 6000 50  0001 C CNN
 	1    1500 6000
