File: doc/kicad/fmdp-1-b/FMDP-1-B/FMDP-1-B.kicad_pcb (KiCad board)
At the start: 2 copper layers, 0 parts

Commit message: doc/kicad: FMDP-1-B v0.1
Parts:
- added C1: 0.1u 100V, Capacitor_SMD:C_0805_2012Metric, B.Cu at (36.5, 46.5)
- added C2: 10u 25V, Capacitor_SMD:C_0805_2012Metric, B.Cu at (38.5, 44.0)
- added C3: 0.1u 100V, Capacitor_SMD:C_0805_2012Metric, B.Cu at (46.5, 67.5)
- added C4: 10u 25V, Capacitor_SMD:C_0805_2012Metric, B.Cu at (44.5, 70.0)
- added D1: LED, LED_SMD:LED_0402_1005Metric, F.Cu at (34.0, 53.0)
- added D2: LED, LED_SMD:LED_0402_1005Metric, F.Cu at (49.0, 61.0)
- added J1: Conn_01x01, fmlibf:JS-2x2mm, F.Cu at (43.1, 33.1)
- added J2: Conn_01x01, fmlibf:JS-2x2mm, F.Cu at (34.1, 33.1)
- added J3: Conn_01x01, fmlibf:JS-2x2mm, F.Cu at (39.9, 80.9)
- added J4: Conn_01x01, fmlibf:JS-2x2mm, F.Cu at (48.9, 80.9)
- added JC1: Conn_01x01, fmlibf:JS-1x2mm, F.Cu at (44.5, 46.5)
- added JC2: Conn_01x01, fmlibf:JS-1x2mm, F.Cu at (44.5, 48.0)
- added JC3: Conn_01x01, fmlibf:JS-1x2mm, F.Cu at (38.5, 67.5)
- added JC4: Conn_01x01, fmlibf:JS-1x2mm, F.Cu at (38.5, 66.0)
- added JG1: Conn_01x01, fmlibf:JS-2x2mm, F.Cu at (48.9, 43.7)
- added JG2: Conn_01x01, fmlibf:JS-2x2mm, F.Cu at (34.1, 70.3)
- added JL1: Conn_01x01, fmlibf:JS-1x2mm, B.Cu at (34.0, 55.0)
- added JL2: Conn_01x01, fmlibf:JS-1x2mm, B.Cu at (49.0, 59.0)
- added JP1: Conn_01x01, fmlibf:JS-2x2mm, B.Cu at (37.5, 42.0)
- added JP2: Conn_01x01, fmlibf:JS-2x2mm, B.Cu at (45.5, 72.0)
- added JS11: Conn_01x01, fmlibf:JS-1x2mm, F.Cu at (36.5, 51.0)
- added JS12: Conn_01x01, fmlibf:JS-1x2mm, F.Cu at (36.5, 55.0)
- added JS13: Conn_01x01, fmlibf:JS-1x2mm, F.Cu at (39.0, 51.0)
- added JS14: Conn_01x01, fmlibf:JS-1x2mm, F.Cu at (39.0, 55.0)
- added JS15: Conn_01x01, fmlibf:JS-1x2mm, F.Cu at (41.5, 51.0)
- added JS16: Conn_01x01, fmlibf:JS-1x2mm, F.Cu at (41.5, 55.0)
- added JS17: Conn_01x01, fmlibf:JS-1x2mm, F.Cu at (44.0, 51.0)
- added JS18: Conn_01x01, fmlibf:JS-1x2mm, F.Cu at (44.0, 55.0)
- added JS21: Conn_01x01, fmlibf:JS-1x2mm, F.Cu at (46.5, 63.0)
- added JS22: Conn_01x01, fmlibf:JS-1x2mm, F.Cu at (46.5, 59.0)
- added JS23: Conn_01x01, fmlibf:JS-1x2mm, F.Cu at (44.0, 63.0)
- added JS24: Conn_01x01, fmlibf:JS-1x2mm, F.Cu at (44.0, 59.0)
- added JS25: Conn_01x01, fmlibf:JS-1x2mm, F.Cu at (41.5, 63.0)
- added JS26: Conn_01x01, fmlibf:JS-1x2mm, F.Cu at (41.5, 59.0)
- added JS27: Conn_01x01, fmlibf:JS-1x2mm, F.Cu at (39.0, 63.0)
- added JS28: Conn_01x01, fmlibf:JS-1x2mm, F.Cu at (39.0, 59.0)
- added JV1: Conn_01x01, fmlibf:JS-1x2mm, F.Cu at (34.0, 55.0)
- added JV2: Conn_01x01, fmlibf:JS-1x2mm, F.Cu at (49.0, 59.0)
- added Q1: AOD482, Package_TO_SOT_SMD:TO-252-2, F.Cu at (47.0, 37.4)
- added Q2: AOD482, Package_TO_SOT_SMD:TO-252-2, F.Cu at (38.0, 37.4)
- added Q3: AOD482, Package_TO_SOT_SMD:TO-252-2, F.Cu at (36.0, 76.6)
- added Q4: AOD482, Package_TO_SOT_SMD:TO-252-2, F.Cu at (45.0, 76.6)
- added R1: 100?, Resistor_SMD:R_0402_1005Metric, B.Cu at (34.0, 53.0)
- added R11: 3.3k, Resistor_SMD:R_0402_1005Metric, B.Cu at (36.5, 53.0)
- added R12: 100k, Resistor_SMD:R_0402_1005Metric, F.Cu at (36.5, 53.0)
- added R13: 4.7k, Resistor_SMD:R_0402_1005Metric, B.Cu at (39.0, 53.0)
- added R14: 3.3k, Resistor_SMD:R_0402_1005Metric, F.Cu at (39.0, 53.0)
- added R15: 4.7k, Resistor_SMD:R_0402_1005Metric, B.Cu at (41.5, 53.0)
- added R16: 3.3k, Resistor_SMD:R_0402_1005Metric, F.Cu at (41.5, 53.0)
- added R17: 4.7k, Resistor_SMD:R_0402_1005Metric, B.Cu at (44.0, 53.0)
- added R18: 3.3k, Resistor_SMD:R_0402_1005Metric, F.Cu at (44.0, 53.0)
- added R2: 100?, Resistor_SMD:R_0402_1005Metric, B.Cu at (49.0, 61.0)
- added R21: 3.3k, Resistor_SMD:R_0402_1005Metric, B.Cu at (46.5, 61.0)
- added R22: 100k, Resistor_SMD:R_0402_1005Metric, F.Cu at (46.5, 61.0)
- added R23: 4.7k, Resistor_SMD:R_0402_1005Metric, B.Cu at (44.0, 61.0)
- added R24: 3.3k, Resistor_SMD:R_0402_1005Metric, F.Cu at (44.0, 61.0)
- added R25: 4.7k, Resistor_SMD:R_0402_1005Metric, B.Cu at (41.5, 61.0)
- added R26: 3.3k, Resistor_SMD:R_0402_1005Metric, F.Cu at (41.5, 61.0)
- added R27: 4.7k, Resistor_SMD:R_0402_1005Metric, B.Cu at (39.0, 61.0)
- added R28: 3.3k, Resistor_SMD:R_0402_1005Metric, F.Cu at (39.0, 61.0)
- added U1: UCC27211, Package_SO:SOIC-8-1EP_3.9x4.9mm_P1.27mm_EP2.29x3mm, F.Cu at (40.0, 46.0)
- added U2: UCC27211, Package_SO:SOIC-8-1EP_3.9x4.9mm_P1.27mm_EP2.29x3mm, F.Cu at (43.0, 68.0)
Routing:
- net /B1/HS: track 0.00 -> 25.8 mm, vias 0 -> 2
- net /B2/HS: track 0.00 -> 25.7 mm, vias 0 -> 2
- net /B2/HO: track 0.00 -> 7.04 mm
- net /B1/HO: track 0.00 -> 7.04 mm
- net /B2/LO: track 0.00 -> 3.40 mm
- net /B1/LO: track 0.00 -> 3.34 mm
- net /B2/HI: track 0.00 -> 1.93 mm
- net /B1/HI: track 0.00 -> 1.93 mm
- net /B1/LI: track 0.00 -> 1.89 mm
- net /B2/LI: track 0.00 -> 1.79 mm
- net Net-(C1-Pad1): track 0.00 -> 1.76 mm, vias 0 -> 1
- net Net-(C3-Pad1): track 0.00 -> 1.76 mm, vias 0 -> 1
- net /B2/VH: track 0.00 -> 1.70 mm
- net /B1/VH: track 0.00 -> 1.70 mm
- net Net-(JS28-Pad1): track 0.00 -> 1.50 mm
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- added copper zone on B.Cu, net GND
- added copper zone on F.Cu, net GND
Other:
- board outline added: 17 x 50 mm
- board text added: "2020-12-30"
- board text added: "FMDP-1-B v0.1"
